File: czujnik.kicad_sch (KiCad schematic)
At the start: 9 parts, among them J4 Conn IN, J5 Conn OUT, U4 BME280, U5 MB85RS256B

Commit message: awetg
Parts:
- removed J4: Conn IN, Connector_PinHeader_2.54mm:PinHeader_2x09_P2.54mm_Vertical, symbol Connector_Generic:Conn_02x09_Odd_Even
- removed J5: Conn OUT, Connector_PinSocket_2.54mm:PinSocket_2x09_P2.54mm_Vertical, symbol Connector_Generic:Conn_02x09_Odd_Even
- added J4: Conn_01x08, Connector_PinHeader_2.54mm:PinHeader_1x08_P2.54mm_Vertical, symbol Connector_Generic:Conn_01x08
- added J5: Conn_01x10, Connector_PinHeader_2.54mm:PinHeader_1x10_P2.54mm_Vertical, symbol Connector_Generic:Conn_01x10
- renumbered U4 to U5, U5 to U6
Connections:
- net +3.3V: now also J4.1 (Pin_1)
- net COL 1: now also J5.1 (Pin_1)
- net COL 2: now also J5.2 (Pin_2)
- net COL 3: now also J5.3 (Pin_3)
- net COL 4: now also J5.4 (Pin_4)
- net CS BME280: now also J4.2 (Pin_2)
- net CS FRAM SPI: now also J4.3 (Pin_3)
- net GND: now also J5.10 (Pin_10), J5.9 (Pin_9)
- net MISO: now also J4.5 (Pin_5)
- net MOSI: now also J4.4 (Pin_4)
- net ROW 1: now also J5.5 (Pin_5)
- net ROW 2: now also J5.6 (Pin_6)
- net ROW 3: now also J5.7 (Pin_7)
- net ROW 4: now also J5.8 (Pin_8)
- net SCK: now also J4.6 (Pin_6)
- net SCL: now also J4.8 (Pin_8)
- net SDA: now also J4.7 (Pin_7)
