File: klawiaturka.kicad_sch (KiCad schematic)
At the start: 0 parts

Commit message: Test
Parts:
- added D1, D2, D3, D4: D_Schottky, Diode_SMD:D_SMA, symbol Device:D_Schottky
- added J8: Conn_K, symbol Connector_Generic:Conn_02x04_Counter_Clockwise
- added SW1, SW10, SW11, SW12, SW13, SW14, SW15, SW16, SW17, SW3, SW4, SW5, SW6, SW7, SW8, SW9: SW_Push, Button_Switch_SMD:SW_SPST_Omron_B3FS-100xP, symbol Switch:SW_Push
Connections:
- new net: D3.2 (A), SW12.2, SW16.2, SW6.2, SW8.2
- new net: D2.2 (A), SW11.2, SW15.2, SW4.2, SW5.2
- new net: D4.2 (A), SW13.2, SW17.2, SW7.2, SW9.2
- new net: D1.2 (A), SW1.2, SW10.2, SW14.2, SW3.2
- new net COL 1: D1.1 (K), J8.8 (Pin_8)
- new net COL 2: D2.1 (K), J8.7 (Pin_7)
- new net COL 3: D3.1 (K), J8.6 (Pin_6)
- new net COL 4: D4.1 (K), J8.5 (Pin_5)
- new net ROW 1: J8.1 (Pin_1), SW1.1, SW5.1, SW6.1, SW7.1
- new net ROW 2: J8.2 (Pin_2), SW3.1, SW4.1, SW8.1, SW9.1
- new net ROW 3: J8.3 (Pin_3), SW10.1, SW11.1, SW12.1, SW13.1
- new net ROW 4: J8.4 (Pin_4), SW14.1, SW15.1, SW16.1, SW17.1

Commit message: Orange 21.37
Parts:
- removed J8: Conn_K, symbol Connector_Generic:Conn_02x04_Counter_Clockwise
- added J6: Conn, symbol Connector_Generic:Conn_02x09_Odd_Even
Connections:
- net COL 1: now also J6.2 (Pin_2)
- net COL 2: now also J6.4 (Pin_4)
- net COL 3: now also J6.6 (Pin_6)
- net COL 4: now also J6.8 (Pin_8)
- net ROW 1: now also J6.16 (Pin_16)
- net ROW 2: now also J6.14 (Pin_14)
- net ROW 3: now also J6.12 (Pin_12)
- net ROW 4: now also J6.10 (Pin_10)

Commit message: małe zmiany poprawki dsagolih
Parts:
- renumbered SW15 to SW10, SW6 to SW11, SW8 to SW12, SW12 to SW13, SW16 to SW14, SW7 to SW15, SW9 to SW16, SW13 to SW17, SW17 to SW18, SW1 to SW3, SW3 to SW4, SW10 to SW5, SW14 to SW6, SW5 to SW7, SW4 to SW8, SW11 to SW9
Connections:
- no-connect marks 0 -> 10
Changed lines of the file:
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@@
 		(color 0 0 0 0)
 	)
+	(no_connect
+		(at 195.58 63.5)
+	)
+	(no_connect
+		(at 195.58 71.12)
+	)
+	(no_connect
+		(at 195.58 55.88)
+	)
+	(no_connect
+		(at 195.58 53.34)
+	)
+	(no_connect
+		(at 195.58 68.58)
+	)
+	(no_connect
+		(at 210.82 73.66)
+	)
+	(no_connect
+		(at 195.58 66.04)
+	)
+	(no_connect
+		(at 195.58 60.96)
+	)
+	(no_connect
+		(at 195.58 73.66)
+	)
+	(no_connect
+		(at 195.58 58.42)
+	)
 	(wire
 		(pts
@@
 	(wire
 		(pts
+			(xy 195.58 66.04) (xy 196.85 66.04)
+		)
+		(stroke
+			(width 0)
+			(type default)
+		)
+	)
+	(wire
+		(pts
 			(xy 99.06 116.84) (xy 100.33 116.84)
 		)
@@
 	(wire
 		(pts
+			(xy 195.58 58.42) (xy 196.85 58.42)
+		)
+		(stroke
+			(width 0)
+			(type default)
+		)
+	)
+	(wire
+		(pts
 			(xy 99.06 116.84) (xy 99.06 120.65)
 		)
@@
 	(wire
 		(pts
+			(xy 195.58 71.12) (xy 196.85 71.12)
+		)
+		(stroke
+			(width 0)
+			(type default)
+		)
+	)
+	(wire
+		(pts
 			(xy 92.71 116.84) (xy 92.71 132.08)
 		)
@@
 	(wire
 		(pts
+			(xy 195.58 53.34) (xy 196.85 53.34)
+		)
+		(stroke
+			(width 0)
+			(type default)
+		)
+	)
+	(wire
+		(pts
 			(xy 78.74 116.84) (xy 78.74 120.65)
 		)
@@
 	(wire
 		(pts
+			(xy 210.82 73.66) (xy 209.55 73.66)
+		)
+		(stroke
+			(width 0)
+			(type default)
+		)
+	)
+	(wire
+		(pts
 			(xy 92.71 87.63) (xy 92.71 101.6)
 		)
@@
 	(wire
 		(pts
+			(xy 195.58 55.88) (xy 196.85 55.88)
+		)
+		(stroke
+			(width 0)
+			(type default)
+		)
+	)
+	(wire
+		(pts
 			(xy 74.93 120.65) (xy 78.74 120.65)
 		)
@@
 	(wire
 		(pts
+			(xy 195.58 60.96) (xy 196.85 60.96)
+		)
+		(stroke
+			(width 0)
+			(type default)
+		)
+	)
+	(wire
+		(pts
 			(xy 209.55 55.88) (xy 212.09 55.88)
 		)
@@
 	(wire
 		(pts
+			(xy 195.58 73.66) (xy 196.85 73.66)
+		)
+		(stroke
+			(width 0)
+			(type default)
+		)
+	)
+	(wire
+		(pts
 			(xy 152.4 132.08) (xy 153.67 132.08)
 		)
@@
 	(wire
 		(pts
+			(xy 195.58 68.58) (xy 196.85 68.58)
+		)
+		(stroke
+			(width 0)
+			(type default)
+		)
+	)
+	(wire
+		(pts
 			(xy 212.09 63.5) (xy 209.55 63.5)
 		)
@@
 		(pts
 			(xy 99.06 147.32) (xy 100.33 147.32)
+		)
+		(stroke
+			(width 0)
+			(type default)
+		)
+	)
+	(wire
+		(pts
+			(xy 195.58 63.5) (xy 196.85 63.5)
 		)
 		(stroke
@@
 		(dnp no)
 		(fields_autoplaced yes)
-		(property "Reference" "SW8"
+		(property "Reference" "SW12"
 			(at 125.73 109.22 0)
 			(show_name no)
@@
 			(project "Projekt_smiw"
 				(path "/632074d6-5d6d-4a29-990c-0b192b6b381d"
-					(reference "SW8")
+					(reference "SW12")
 					(unit 1)
 				)
@@
 		(dnp no)
 		(fields_autoplaced yes)
-		(property "Reference" "SW4"
+		(property "Reference" "SW8"
 			(at 105.41 109.22 0)
 			(show_name no)
@@
 			(project "Projekt_smiw"
 				(path "/632074d6-5d6d-4a29-990c-0b192b6b381d"
-					(reference "SW4")
+					(reference "SW8")
 					(unit 1)
 				)
@@
 		(dnp no)
 		(fields_autoplaced yes)
-		(property "Reference" "SW6"
+		(property "Reference" "SW11"
 			(at 125.73 93.98 0)
 			(show_name no)
@@
 			(project "Projekt_smiw"
 				(path "/632074d6-5d6d-4a29-990c-0b192b6b381d"
-					(reference "SW6")
+					(reference "SW11")
 					(unit 1)
 				)
@@
 		(dnp no)
 		(fields_autoplaced yes)
-		(property "Reference" "SW7"
+		(property "Reference" "SW15"
 			(at 146.05 93.98 0)
 			(show_name no)
@@
 			(project "Projekt_smiw"
 				(path "/632074d6-5d6d-4a29-990c-0b192b6b381d"
-					(reference "SW7")
+					(reference "SW15")
 					(unit 1)
 				)
@@
 		(dnp no)
 		(fields_autoplaced yes)
-		(property "Reference" "SW14"
+		(property "Reference" "SW6"
 			(at 85.09 139.7 0)
 			(show_name no)
@@
 			(project "Projekt_smiw"
 				(path "/632074d6-5d6d-4a29-990c-0b192b6b381d"
-					(reference "SW14")
+					(reference "SW6")
 					(unit 1)
 				)
@@
 		(dnp no)
 		(fields_autoplaced yes)
-		(property "Reference" "SW1"
+		(property "Reference" "SW3"
 			(at 85.09 93.98 0)
 			(show_name no)
@@
 			(project "Projekt_smiw"
 				(path "/632074d6-5d6d-4a29-990c-0b192b6b381d"
-					(reference "SW1")
+					(reference "SW3")
 					(unit 1)
 				)
@@
 		(dnp no)
 		(fields_autoplaced yes)
-		(property "Reference" "SW11"
+		(property "Reference" "SW9"
 			(at 105.41 124.46 0)
 			(show_name no)
@@
 			(project "Projekt_smiw"
 				(path "/632074d6-5d6d-4a29-990c-0b192b6b381d"
-					(reference "SW11")
+					(reference "SW9")
 					(unit 1)
 				)
@@
 		(dnp no)
 		(fields_autoplaced yes)
-		(property "Reference" "SW9"
+		(property "Reference" "SW16"
 			(at 147.32 109.22 0)
 			(show_name no)
@@
 			(project "Projekt_smiw"
 				(path "/632074d6-5d6d-4a29-990c-0b192b6b381d"
-					(reference "SW9")
+					(reference "SW16")
 					(unit 1)
 				)
@@
 		(dnp no)
 		(fields_autoplaced yes)
-		(property "Reference" "SW10"
+		(property "Reference" "SW5"
 			(at 85.09 124.46 0)
 			(show_name no)
@@
 			(project "Projekt_smiw"
 				(path "/632074d6-5d6d-4a29-990c-0b192b6b381d"
-					(reference "SW10")
+					(reference "SW5")
 					(unit 1)
 				)
@@
 		(dnp no)
 		(fields_autoplaced yes)
-		(property "Reference" "SW3"
+		(property "Reference" "SW4"
 			(at 85.09 109.22 0)
 			(show_name no)
@@
 			(project "Projekt_smiw"
 				(path "/632074d6-5d6d-4a29-990c-0b192b6b381d"
-					(reference "SW3")
+					(reference "SW4")
 					(unit 1)
 				)
@@
 		(dnp no)
 		(fields_autoplaced yes)
-		(property "Reference" "SW12"
+		(property "Reference" "SW13"
 			(at 125.73 124.46 0)
 			(show_name no)
@@
 			(project "Projekt_smiw"
 				(path "/632074d6-5d6d-4a29-990c-0b192b6b381d"
-					(reference "SW12")
+					(reference "SW13")
 					(unit 1)
 				)
@@
 		(dnp no)
 		(fields_autoplaced yes)
-		(property "Reference" "SW5"
+		(property "Reference" "SW7"
 			(at 105.41 93.98 0)
 			(show_name no)
@@
 			(project "Projekt_smiw"
 				(path "/632074d6-5d6d-4a29-990c-0b192b6b381d"
-					(reference "SW5")
+					(reference "SW7")
 					(unit 1)
 				)
@@
 		(dnp no)
 		(fields_autoplaced yes)
-		(property "Reference" "SW15"
+		(property "Reference" "SW10"
 			(at 105.41 139.7 0)
 			(show_name no)
@@
 			(project "Projekt_smiw"
 				(path "/632074d6-5d6d-4a29-990c-0b192b6b381d"
-					(reference "SW15")
+					(reference "SW10")
 					(unit 1)
 				)
@@
 		(dnp no)
 		(fields_autoplaced yes)
-		(property "Reference" "SW16"
+		(property "Reference" "SW14"
 			(at 125.73 139.7 0)
 			(show_name no)
@@
 			(project "Projekt_smiw"
 				(path "/632074d6-5d6d-4a29-990c-0b192b6b381d"
-					(reference "SW16")
+					(reference "SW14")
 					(unit 1)
 				)
@@
 		(dnp no)
 		(fields_autoplaced yes)
-		(property "Reference" "SW13"
+		(property "Reference" "SW17"
 			(at 147.32 124.46 0)
 			(show_name no)
@@
 			(project "Projekt_smiw"
 				(path "/632074d6-5d6d-4a29-990c-0b192b6b381d"
-					(reference "SW13")
+					(reference "SW17")
 					(unit 1)
 				)
@@
 		(dnp no)
 		(fields_autoplaced yes)
-		(property "Reference" "SW17"
+		(property "Reference" "SW18"
 			(at 147.32 139.7 0)
 			(show_name no)
@@
 			(project "Projekt_smiw"
 				(path "/632074d6-5d6d-4a29-990c-0b192b6b381d"
-					(reference "SW17")
+					(reference "SW18")
 					(unit 1)
 				)

Commit message: footprinty all, aheoi;rthipoawert;hiogsedho;i yay Halo? Schemat zrobiony ^^ pewnie nie
Parts:
- added J7: Conn OUT, Connector_PinSocket_2.54mm:PinSocket_2x09_P2.54mm_Vertical, symbol Connector_Generic:Conn_02x09_Odd_Even
- D1, D2, D3, D4: footprint Diode_SMD:D_SMA -> Diode_SMD:D_0603_1608Metric
- J6: value Conn -> Conn IN; footprint (none) -> Connector_PinHeader_2.54mm:PinHeader_2x09_P2.54mm_Vertical
Connections:
- net COL 1: now also J7.2 (Pin_2)
- net COL 2: now also J7.4 (Pin_4)
- net COL 3: now also J7.6 (Pin_6)
- net COL 4: now also J7.8 (Pin_8)
- net ROW 1: now also J6.10 (Pin_10), J7.10 (Pin_10); no longer J6.16 (Pin_16)
- net ROW 2: now also J6.12 (Pin_12), J7.12 (Pin_12); no longer J6.14 (Pin_14)
- net ROW 3: now also J6.14 (Pin_14), J7.14 (Pin_14); no longer J6.12 (Pin_12)
- net ROW 4: now also J6.16 (Pin_16), J7.16 (Pin_16); no longer J6.10 (Pin_10)
- net +3.3V: now reaches J6.1 (Pin_1)
- net +3.3V: now also J7.1 (Pin_1)
- net SCK: now reaches J6.11 (Pin_11)
- net SCK: now also J7.11 (Pin_11)
- net SDA: now reaches J6.13 (Pin_13)
- net SDA: now also J7.13 (Pin_13)
- net SCL: now reaches J6.15 (Pin_15)
- net SCL: now also J7.15 (Pin_15)
- net GND: now reaches J6.17 (Pin_17)
- net GND: now also J6.18 (Pin_18), J7.17 (Pin_17), J7.18 (Pin_18)
- net CS BME280: now reaches J6.3 (Pin_3)
- net CS BME280: now also J7.3 (Pin_3)
- net CS FRAM SPI: now reaches J6.5 (Pin_5)
- net CS FRAM SPI: now also J7.5 (Pin_5)
- net MOSI: now reaches J6.7 (Pin_7)
- net MOSI: now also J7.7 (Pin_7)
- net MISO: now reaches J6.9 (Pin_9)
- net MISO: now also J7.9 (Pin_9)
- no-connect marks 10 -> 0

Commit message: awetg
Parts:
- removed J6: Conn IN, Connector_PinHeader_2.54mm:PinHeader_2x09_P2.54mm_Vertical, symbol Connector_Generic:Conn_02x09_Odd_Even
- removed J7: Conn OUT, Connector_PinSocket_2.54mm:PinSocket_2x09_P2.54mm_Vertical, symbol Connector_Generic:Conn_02x09_Odd_Even
- added J6: Conn_01x08, Connector_PinHeader_2.54mm:PinHeader_1x08_P2.54mm_Vertical, symbol Connector_Generic:Conn_01x08
- added J7: Conn_01x10, Connector_PinHeader_2.54mm:PinHeader_1x10_P2.54mm_Vertical, symbol Connector_Generic:Conn_01x10
Connections:
- net +3.3V: now also J6.1 (Pin_1)
- net COL 1: now also J7.1 (Pin_1)
- net COL 2: now also J7.2 (Pin_2)
- net COL 3: now also J7.3 (Pin_3)
- net COL 4: now also J7.4 (Pin_4)
- net CS BME280: now also J6.2 (Pin_2)
- net CS FRAM SPI: now also J6.3 (Pin_3)
- net GND: now also J7.10 (Pin_10), J7.9 (Pin_9)
- net MISO: now also J6.5 (Pin_5)
- net MOSI: now also J6.4 (Pin_4)
- net ROW 1: now also J7.5 (Pin_5)
- net ROW 2: now also J7.6 (Pin_6)
- net ROW 3: now also J7.7 (Pin_7)
- net ROW 4: now also J7.8 (Pin_8)
- net SCK: now also J6.6 (Pin_6)
- net SCL: now also J6.8 (Pin_8)
- net SDA: now also J6.7 (Pin_7)
