File: Projekt_smiw.kicad_pcb (KiCad board)
At the start: 2 copper layers, 63 parts, among them J1 USB_C_Receptacle_USB2.0, J2 Conn OUT, J4 Conn IN, J5 Conn OUT, J6 Conn IN, J7 Conn OUT, J8 Conn IN, SW1 SW_Omron_B3FS, SW10 SW_Push, SW11 SW_Push, SW12 SW_Push, SW13 SW_Push, SW14 SW_Push, SW15 SW_Push, SW16 SW_Push, SW17 SW_Push, SW18 SW_Push, SW2 SW_Omron_B3FS, SW3 SW_Push, SW4 SW_Push, SW5 SW_Push, SW6 SW_Push, SW7 SW_Push, SW8 SW_Push, SW9 SW_Push, U1 USBLC6-2P6, U2 NCP1117-3.3_SOT223, U3 ESP32-S3-PICO-1, U4 BME280, U5 MB85RS256B, U6 MB85RC256V, U7 SSD1306, U8 LM1117DT-3.3

Commit message: awetg
Parts:
- removed C16: 10μF, Capacitor_SMD:C_0805_2012Metric
- added C1: 10μF, Capacitor_SMD:C_0805_2012Metric, F.Cu at (195.7, 116.5)
- added J3: Conn_01x10, Connector_PinSocket_2.54mm:PinSocket_1x10_P2.54mm_Vertical, F.Cu at (180.0, 89.8)
- added J9: Conn_01x10, Connector_PinHeader_2.54mm:PinHeader_1x10_P2.54mm_Vertical, F.Cu at (199.0, 89.8)
- J2: value Conn OUT -> Conn_01x08; footprint Connector_PinSocket_2.54mm:PinSocket_2x09_P2.54mm_Vertical -> Connector_PinSocket_2.54mm:PinSocket_1x08_P2.54mm_Vertical
- J4, J6, J8: value Conn IN -> Conn_01x08; footprint Connector_PinHeader_2.54mm:PinHeader_2x09_P2.54mm_Vertical -> Connector_PinHeader_2.54mm:PinHeader_1x08_P2.54mm_Vertical
- J5, J7: value Conn OUT -> Conn_01x10; footprint Connector_PinSocket_2.54mm:PinSocket_2x09_P2.54mm_Vertical -> Connector_PinHeader_2.54mm:PinHeader_1x10_P2.54mm_Vertical
- U3: value ESP32-S3-PICO-1 -> LM1117DT-3.3; footprint Package_DFN_QFN:QFN-56-1EP_7x7mm_P0.4mm_EP4x4mm -> Package_TO_SOT_SMD:TO-252-3_TabPin2
- U4: value BME280 -> ESP32-S3-PICO-1; footprint Package_LGA:Bosch_LGA-8_2.5x2.5mm_P0.65mm_ClockwisePinNumbering -> Package_DFN_QFN:QFN-56-1EP_7x7mm_P0.4mm_EP4x4mm
- U5: value MB85RS256B -> BME280; footprint Package_SO:SOIC-8_3.9x4.9mm_P1.27mm -> Package_LGA:Bosch_LGA-8_2.5x2.5mm_P0.65mm_ClockwisePinNumbering
- U6: value MB85RC256V -> MB85RS256B
- U7: value SSD1306 -> MB85RC256V; footprint Display:ER_OLEDM0.91_1x-I2C -> Package_SO:SOIC-8_3.9x4.9mm_P1.27mm
- U8: value LM1117DT-3.3 -> SSD1306; footprint Package_TO_SOT_SMD:TO-252-3_TabPin2 -> Display:ER_OLEDM0.91_1x-I2C
- moved U7 73.3 mm to (186.8, 152.1)
- moved C15 70.0 mm to (192.6, 128.3)
- moved C2 70.0 mm to (184.6, 128.3)
- moved C3 70.0 mm to (184.6, 130.8)
- moved C5 70.0 mm to (184.6, 133.3)
- moved C6 70.0 mm to (184.6, 135.8)
- moved C7 70.0 mm to (184.6, 138.3)
- moved C8 70.0 mm to (184.6, 140.9)
- moved R1 70.0 mm to (192.6, 130.8)
- moved R10 70.0 mm to (196.6, 138.3)
- moved R11 70.0 mm to (196.6, 140.9)
- moved R2 70.0 mm to (192.6, 133.3)
- moved R3 70.0 mm to (192.6, 135.8)
- moved R4 70.0 mm to (192.6, 138.3)
- moved R5 70.0 mm to (192.6, 140.9)
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Connections:
- J2 pad 2: /Root/COL 1 -> /Root/CS BME280
- J2 pad 3: /Root/CS BME280 -> /Root/CS FRAM SPI
- J2 pad 4: /Root/COL 2 -> /Root/MOSI
- J2 pad 5: /Root/CS FRAM SPI -> /Root/MISO
- J2 pad 6: /Root/COL 3 -> /Root/SCK
- J2 pad 7: /Root/MOSI -> /Root/SDA
- J2 pad 8: /Root/COL 4 -> /Root/SCL
- J4 pad 2: /czujnik/COL 1 -> /czujnik/CS BME280
- J4 pad 3: /czujnik/CS BME280 -> /czujnik/CS FRAM SPI
- J4 pad 4: /czujnik/COL 2 -> /czujnik/MOSI
- J4 pad 5: /czujnik/CS FRAM SPI -> /czujnik/MISO
- J4 pad 6: /czujnik/COL 3 -> /czujnik/SCK
- J4 pad 7: /czujnik/MOSI -> /czujnik/SDA
- J4 pad 8: /czujnik/COL 4 -> /czujnik/SCL
- J5 pad 1: +3.3V -> /czujnik/COL 1
- J5 pad 10: /czujnik/ROW 1 -> GND
- J5 pad 2: /czujnik/COL 1 -> /czujnik/COL 2
- J5 pad 3: /czujnik/CS BME280 -> /czujnik/COL 3
- J5 pad 4: /czujnik/COL 2 -> /czujnik/COL 4
- J5 pad 5: /czujnik/CS FRAM SPI -> /czujnik/ROW 1
- J5 pad 6: /czujnik/COL 3 -> /czujnik/ROW 2
- J5 pad 7: /czujnik/MOSI -> /czujnik/ROW 3
- J5 pad 8: /czujnik/COL 4 -> /czujnik/ROW 4
- J5 pad 9: /czujnik/MISO -> GND
- J6 pad 2: /klawiaturka/COL 1 -> /klawiaturka/CS BME280
- J6 pad 3: /klawiaturka/CS BME280 -> /klawiaturka/CS FRAM SPI
- J6 pad 4: /klawiaturka/COL 2 -> /klawiaturka/MOSI
- J6 pad 5: /klawiaturka/CS FRAM SPI -> /klawiaturka/MISO
- J6 pad 6: /klawiaturka/COL 3 -> /klawiaturka/SCK
- J6 pad 7: /klawiaturka/MOSI -> /klawiaturka/SDA
- J6 pad 8: /klawiaturka/COL 4 -> /klawiaturka/SCL
- J7 pad 1: +3.3V -> /klawiaturka/COL 1
- J7 pad 10: /klawiaturka/ROW 1 -> GND
- J7 pad 2: /klawiaturka/COL 1 -> /klawiaturka/COL 2
- J7 pad 3: /klawiaturka/CS BME280 -> /klawiaturka/COL 3
- J7 pad 4: /klawiaturka/COL 2 -> /klawiaturka/COL 4
- J7 pad 5: /klawiaturka/CS FRAM SPI -> /klawiaturka/ROW 1
- J7 pad 6: /klawiaturka/COL 3 -> /klawiaturka/ROW 2
- J7 pad 7: /klawiaturka/MOSI -> /klawiaturka/ROW 3
- J7 pad 8: /klawiaturka/COL 4 -> /klawiaturka/ROW 4
- J7 pad 9: /klawiaturka/MISO -> GND
- J8 pad 2: /wyświetlacz/COL 1 -> /wyświetlacz/CS BME280
- J8 pad 3: /wyświetlacz/CS BME280 -> /wyświetlacz/CS FRAM SPI
- J8 pad 4: /wyświetlacz/COL 2 -> /wyświetlacz/MOSI
- J8 pad 5: /wyświetlacz/CS FRAM SPI -> /wyświetlacz/MISO
- J8 pad 6: /wyświetlacz/COL 3 -> /wyświetlacz/SCK
- J8 pad 7: /wyświetlacz/MOSI -> /wyświetlacz/SDA
- J8 pad 8: /wyświetlacz/COL 4 -> /wyświetlacz/SCL
- R10 pad 1: Net-(U6-A2) -> Net-(U7-A2)
- R11 pad 1: Net-(U6-WP) -> Net-(U7-WP)
- R6 pad 2: Net-(U5-~{HOLD}) -> Net-(U6-~{HOLD})
- R7 pad 2: Net-(U5-~{WP}) -> Net-(U6-~{WP})
- R8 pad 1: Net-(U6-A0) -> Net-(U7-A0)
- R9 pad 1: Net-(U6-A1) -> Net-(U7-A1)
- U3 pad 2: +3.3V -> unconnected-(U3-VO-Pad2)
- U3 pad 3: +3.3V -> unconnected-(U3-VI-Pad3)
- U4 pad 1: GND -> unconnected-(U4-LNA_IN-Pad1)
- U4 pad 2: /czujnik/CS BME280 -> +3.3V
- U4 pad 3: /czujnik/MOSI -> +3.3V
- U4 pad 4: /czujnik/SCK -> /Root/RESET
- U4 pad 5: /czujnik/MISO -> /Root/BOOT
- U4 pad 6: +3.3V -> /Root/CS FRAM SPI
- U4 pad 7: GND -> /Root/CS BME280
- U4 pad 8: +3.3V -> unconnected-(U4-GPIO3-Pad8)
- U5 pad 1: /czujnik/CS FRAM SPI -> GND
- U5 pad 2: /czujnik/MISO -> /czujnik/CS BME280
- U5 pad 3: Net-(U5-~{WP}) -> /czujnik/MOSI
- U5 pad 4: GND -> /czujnik/SCK
- U5 pad 5: /czujnik/MOSI -> /czujnik/MISO
- U5 pad 6: /czujnik/SCK -> +3.3V
- U5 pad 7: Net-(U5-~{HOLD}) -> GND
- U6 pad 1: Net-(U6-A0) -> /czujnik/CS FRAM SPI
- U6 pad 2: Net-(U6-A1) -> /czujnik/MISO
- U6 pad 3: Net-(U6-A2) -> Net-(U6-~{WP})
- U6 pad 5: /wyświetlacz/SDA -> /czujnik/MOSI
- U6 pad 6: /wyświetlacz/SCL -> /czujnik/SCK
- U6 pad 7: Net-(U6-WP) -> Net-(U6-~{HOLD})
- U7 pad 1: GND -> Net-(U7-A0)
- U7 pad 2: +3.3V -> Net-(U7-A1)
- U7 pad 3: /wyświetlacz/SCL -> Net-(U7-A2)
- U7 pad 4: /wyświetlacz/SDA -> GND
- U8 pad 1: unconnected-(U8-GND-Pad1) -> GND
- U8 pad 2: unconnected-(U8-VO-Pad2) -> +3.3V
- U8 pad 3: unconnected-(U8-VI-Pad3) -> /wyświetlacz/SCL

Commit message: PCB project procesor
Parts:
- removed C12, C13, C14, C15: 100nF, Capacitor_SMD:C_0603_1608Metric
- removed D1, D2, D3, D4: D_Schottky, Diode_SMD:D_0603_1608Metric
- removed J4, J6, J8: Conn_01x08, Connector_PinHeader_2.54mm:PinHeader_1x08_P2.54mm_Vertical
- removed J5, J7, J9: Conn_01x10, Connector_PinHeader_2.54mm:PinHeader_1x10_P2.54mm_Vertical
- removed R10, R11, R6, R7, R8, R9: 10k, Resistor_SMD:R_0603_1608Metric
- removed SW10, SW11, SW12, SW13, SW14, SW15, SW16, SW17, SW18, SW3, SW4, SW5, SW6, SW7, SW8, SW9: SW_Push, Button_Switch_SMD:SW_SPST_Omron_B3FS-100xP
- removed U3: LM1117DT-3.3, Package_TO_SOT_SMD:TO-252-3_TabPin2
- removed U5: BME280, Package_LGA:Bosch_LGA-8_2.5x2.5mm_P0.65mm_ClockwisePinNumbering
- removed U6: MB85RS256B, Package_SO:SOIC-8_3.9x4.9mm_P1.27mm
- removed U7: MB85RC256V, Package_SO:SOIC-8_3.9x4.9mm_P1.27mm
- removed U8: SSD1306, Display:ER_OLEDM0.91_1x-I2C
- C10, C11, C7, C8, C9, U1: moved to B.Cu
- moved U4 111.2 mm to (201.7, 57.7), turned to 90 degrees
- moved U2 106.3 mm to (187.0, 49.0)
- moved U1 104.1 mm to (187.7, 54.7)
- moved J2 93.7 mm to (212.0, 47.4)
- moved R5 92.2 mm to (199.3, 48.9), turned to 90 degrees
- moved R2 91.8 mm to (176.2, 43.0), turned to -90 degrees
- moved R4 90.0 mm to (201.8, 48.9), turned to 90 degrees
- moved R1 88.9 mm to (178.5, 43.0), turned to -90 degrees
- moved R3 87.8 mm to (204.3, 48.9), turned to 90 degrees
- moved C8 86.7 mm to (196.7, 55.0), turned to 90 degrees
- moved C3 83.2 mm to (194.5, 48.2), turned to 90 degrees
- moved C11 77.8 mm to (207.2, 57.8), turned to 90 degrees
- moved C7 77.1 mm to (202.2, 63.3)
- moved J1 74.5 mm to (168.6, 47.8), turned to -90 degrees
- moved C2 74.1 mm to (181.8, 54.3), turned to -90 degrees
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Connections:
- net /Root/BOOT renamed /BOOT
- net /Root/COL 1 renamed /COL 1
- net /Root/COL 2 renamed /COL 2
- net /Root/COL 3 renamed /COL 3
- net /Root/COL 4 renamed /COL 4
- net /Root/CS BME280 renamed /CS BME280
- net /Root/CS FRAM SPI renamed /CS FRAM SPI
- net /Root/D+ renamed /D+
- net /Root/D- renamed /D-
- net /Root/MISO renamed /MISO
- net /Root/MOSI renamed /MOSI
- net /Root/RESET renamed /RESET
- net /Root/ROW 1 renamed /ROW 1
- net /Root/ROW 2 renamed /ROW 2
- net /Root/ROW 3 renamed /ROW 3
- net /Root/ROW 4 renamed /ROW 4
- net /Root/SCK renamed /SCK
- net /Root/SCL renamed /SCL
- net /Root/SDA renamed /SDA
- net /Root/USB D+ renamed /USB D+
- net /Root/USB D- renamed /USB D-
Routing:
- net +5V: track 0.00 -> 27.3 mm
- net /BOOT: track 0.00 -> 10.7 mm
- net +3.3V: track 0.00 -> 10.7 mm
- net /RESET: track 0.00 -> 10.5 mm
- net /ROW 4: track 0.00 -> 10.2 mm
- net /ROW 3: track 0.00 -> 9.04 mm
- net /MOSI: track 0.00 -> 8.40 mm
- net /COL 2: track 0.00 -> 7.91 mm
- net /MISO: track 0.00 -> 7.51 mm
- net /SCK: track 0.00 -> 7.13 mm
- net /COL 3: track 0.00 -> 7.04 mm
- net /D+: track 0.00 -> 6.07 mm, vias 0 -> 1
- net /ROW 2: track 0.00 -> 5.99 mm
- net /D-: track 0.00 -> 4.42 mm, vias 0 -> 1
- net /ROW 1: track 0.00 -> 3.85 mm
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- added copper zone on F.Cu, net GND
Other:
- board outline added: 53 x 33 mm
- copper layers 2 -> 4

Commit message: pvcv1
Parts:
- R1, R2: moved to B.Cu
- moved R5 14.1 mm to (195.8, 62.5), turned to -90 degrees
- moved R4 13.7 mm to (214.8, 53.4)
- moved R3 10.4 mm to (214.8, 49.1), turned to -90 degrees
- moved R1 6.97 mm to (176.2, 49.6), turned to 180 degrees
- moved R2 3.60 mm to (176.2, 46.6), turned to 180 degrees
- moved C4 2.79 mm to (194.5, 50.0), turned to -90 degrees
- moved C7 2.21 mm to (200.2, 64.2), turned to 90 degrees
- moved C3 2.00 mm to (192.5, 48.2)
- moved C5 2.00 mm to (177.0, 60.7)
- moved C6 2.00 mm to (177.0, 68.5)
- moved SW1 2.00 mm to (171.1, 60.7)
- moved SW2 2.00 mm to (171.0, 68.8)
- moved C9 1.24 mm to (195.8, 59.0)
- moved C8 0.97 mm to (195.8, 55.0)
- moved C10 0.91 mm to (198.6, 64.2), turned to -90 degrees
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Connections:
- J2 pad 2: /CS BME280 -> /SCL
- J2 pad 3: /CS FRAM SPI -> /SDA
- J2 pad 7: /SDA -> /CS BME280
- J2 pad 8: /SCL -> /CS FRAM SPI
Routing:
- net +3.3V: track 10.7 -> 77.3 mm, vias 0 -> 4
- net /BOOT: track 10.7 -> 38.9 mm
- net /RESET: track 10.5 -> 37.2 mm, vias 0 -> 1
- net /USB D-: track 0.00 -> 25.4 mm, vias 0 -> 1
- net /USB D+: track 0.00 -> 24.8 mm, vias 0 -> 1
- net /COL 1: track 0.00 -> 18.2 mm
- net /D-: track 4.42 -> 19.8 mm
- net /SCL: track 0.00 -> 13.5 mm
- net /CS FRAM SPI: track 0.00 -> 13.3 mm, vias 0 -> 1
- net /D+: track 6.07 -> 19.1 mm
- net /CS BME280: track 0.00 -> 11.6 mm, vias 0 -> 1
- net /SDA: track 0.00 -> 11.6 mm
- net /COL 4: track 1.71 -> 12.4 mm
- net GND: track 0.00 -> 8.59 mm, vias 0 -> 1
- net /COL 2: track 7.91 -> 16.3 mm
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- added copper zone on B.Cu, net GND
Other:
- board size 53 x 33 mm -> 55 x 31.5 mm

Commit message: Zmianakonnektorav3
Parts:
- removed J2: Conn_01x08, Connector_PinSocket_2.54mm:PinSocket_1x08_P2.54mm_Vertical
- removed J3: Conn_01x10, Connector_PinSocket_2.54mm:PinSocket_1x10_P2.54mm_Vertical
- added J4: Conn_02x12_Odd_Even, Connector_PinSocket_2.54mm:PinSocket_2x12_P2.54mm_Vertical, F.Cu at (189.7, 40.7)
- added J5: Conn_02x12_Odd_Even, Connector_PinSocket_2.54mm:PinSocket_2x12_P2.54mm_Vertical, F.Cu at (189.7, 68.2)
- U1: moved to F.Cu
- moved J1 55.9 mm to (224.4, 51.2), turned to 90 degrees
- moved C1 46.2 mm to (225.6, 62.0)
- moved C2 44.1 mm to (225.6, 58.6), turned to 90 degrees
- moved R2 40.8 mm to (216.7, 52.4), turned to 0 degrees
- moved R1 40.4 mm to (216.7, 49.4), turned to 0 degrees
- moved U2 35.4 mm to (220.0, 61.8), turned to 180 degrees
- moved R3 33.5 mm to (186.5, 67.2)
- moved R4 33.5 mm to (186.5, 71.5)
- moved U1 29.2 mm to (216.6, 50.9), turned to 180 degrees
- moved C3 26.3 mm to (214.5, 62.6), turned to -90 degrees
- moved C4 21.0 mm to (212.5, 60.9), turned to 90 degrees
Connections:
- U4 pad 21: unconnected-(U4-XTAL_32K_P-Pad21) -> /XTAL_32K_P
- U4 pad 22: unconnected-(U4-XTAL_32K_N-Pad22) -> /XTAL_32K_N
- U4 pad 27: unconnected-(U4-GPIO21-Pad27) -> /GPIO21
- U4 pad 36: unconnected-(U4-SPICLK_N-Pad36) -> /SPICLK_N
- U4 pad 37: unconnected-(U4-SPICLK_P-Pad37) -> /SPICLK_P
- U4 pad 38: unconnected-(U4-GPIO33-Pad38) -> /GPIO33
- U4 pad 39: unconnected-(U4-GPIO34-Pad39) -> /GPIO34
- U4 pad 40: unconnected-(U4-GPIO35-Pad40) -> /GPIO35
- U4 pad 41: unconnected-(U4-GPIO36-Pad41) -> /GPIO36
- U4 pad 42: unconnected-(U4-GPIO37-Pad42) -> /GPIO37
- U4 pad 43: unconnected-(U4-GPIO38-Pad43) -> /GPIO38
- U4 pad 44: unconnected-(U4-MTCK-Pad44) -> /MTCK
- U4 pad 45: unconnected-(U4-MTDO-Pad45) -> /MTDO
- U4 pad 47: unconnected-(U4-MTDI-Pad47) -> /MTDI
- U4 pad 48: unconnected-(U4-MTMS-Pad48) -> /MTMS
- U4 pad 49: unconnected-(U4-U0TXD-Pad49) -> /UOTXD
- U4 pad 50: unconnected-(U4-U0RXD-Pad50) -> /UORXD
- U4 pad 51: unconnected-(U4-GPIO45-Pad51) -> /GPIO45
- U4 pad 52: unconnected-(U4-GPIO46-Pad52) -> /GPIO46
- U4 pad 8: unconnected-(U4-GPIO3-Pad8) -> /GPIO3
Routing:
- net /BOOT: track 38.9 -> 17.6 mm
- net /COL 1: track 18.2 -> 0.00 mm
- net +3.3V: track 77.3 -> 59.3 mm, vias 4 -> 3
- net /COL 2: track 16.3 -> 0.00 mm
- net /D-: track 19.8 -> 4.45 mm, vias 1 -> 0
- net /COL 3: track 14.3 -> 0.00 mm
- net /D+: track 19.1 -> 5.52 mm, vias 1 -> 0
- net /SCL: track 13.5 -> 0.00 mm
- net /CS FRAM SPI: track 13.3 -> 0.00 mm, vias 1 -> 0
- net +5V: track 34.6 -> 22.1 mm, vias 1 -> 0
- net /USB D-: track 25.4 -> 12.9 mm, vias 1 -> 0
- net /COL 4: track 12.4 -> 0.00 mm
- net /USB D+: track 24.8 -> 12.9 mm, vias 1 -> 0
- net /CS BME280: track 11.6 -> 0.00 mm, vias 1 -> 0
- net /SDA: track 11.6 -> 0.00 mm
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Other:
- board size 55 x 31.5 mm -> 66.9 x 38.2 mm

Commit message: Zmianakonnektorav4
Parts:
- moved J5 0.66 mm to (189.7, 68.9)
- moved R3 0.66 mm to (186.5, 67.8)
- moved R4 0.66 mm to (186.5, 72.2)
Routing:
- net +3.3V: track 59.3 -> 31.7 mm
Changed lines of the file:
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@@
 		(tags "CMS SOT")
 		(property "Reference" "U2"
-			(at 0 -4.5 0)
+			(at 0 -5.16 0)
 			(layer "F.SilkS")
 			(effects
@@
 	(footprint "Resistor_SMD:R_0603_1608Metric"
 		(layer "F.Cu")
-		(at 186.5 71.5 90)
+		(at 186.5 72.16 90)
 		(descr "Resistor SMD 0603 (1608 Metric), square (rectangular) end terminal, IPC-7351 nominal, (Body size source: IPC-SM-782 page 72, https://www.pcb-3d.com/wordpress/wp-content/uploads/ipc-sm-782a_amendment_1_and_2.pdf)")
 		(tags "resistor")
@@
 	(footprint "Resistor_SMD:R_0603_1608Metric"
 		(layer "F.Cu")
-		(at 186.5 67.175 -90)
+		(at 186.5 67.835 -90)
 		(descr "Resistor SMD 0603 (1608 Metric), square (rectangular) end terminal, IPC-7351 nominal, (Body size source: IPC-SM-782 page 72, https://www.pcb-3d.com/wordpress/wp-content/uploads/ipc-sm-782a_amendment_1_and_2.pdf)")
 		(tags "resistor")
@@
 	(footprint "Connector_PinSocket_2.54mm:PinSocket_2x12_P2.54mm_Vertical"
 		(layer "F.Cu")
-		(at 189.66 68.2 90)
+		(at 189.66 68.86 90)
 		(descr "Through hole straight socket strip, 2x12, 2.54mm pitch, double rows (from Kicad 4.0.7), script generated")
 		(tags "Through hole socket strip THT 2x12 2.54mm double row")
@@
 		(layer "Edge.Cuts")
 		(pts
-			(xy 220.43083 43.15) (xy 220.43083 68.15)
+			(xy 220.43083 43.81) (xy 220.43083 68.81)
 		)
 		(height 2.4)
@@
 		)
 		(gr_text "25"
-			(at 221.68083 55.65 90)
+			(at 221.68083 56.31 90)
 			(layer "Edge.Cuts")
 			(effects
@@
 	)
 	(segment
-		(start 189.66 70.74)
-		(end 189.66 68.2)
-		(width 0.6)
-		(layer "B.Cu")
-		(net "+3.3V")
-	)
-	(segment
 		(start 206.25 57.875)
 		(end 207.325 57.875)
@@
 		(layer "B.Cu")
 		(net "+3.3V")
-	)
-	(segment
-		(start 189.66 68.2)
-		(end 189.66 43.2)
-		(width 0.6)
-		(layer "B.Cu")
-		(net "+3.3V")

Commit message: poprawkaconnector
Parts:
- moved C6 10.1 mm to (184.0, 61.3)
- moved C5 10.1 mm to (184.0, 53.4)
- moved SW1 10.1 mm to (178.1, 53.4)
- moved SW2 10.1 mm to (178.0, 61.5)
- moved J5 0.20 mm to (189.7, 68.7)
Connections:
- J5 pad 11: /SCK -> /MISO
- J5 pad 13: /CS BME280 -> /MOSI
- J5 pad 15: /CS FRAM SPI -> /SDA
- J5 pad 17: /GPIO3 -> /SCL
- J5 pad 3: /SCL -> /CS FRAM SPI
- J5 pad 5: /SDA -> /CS BME280
- J5 pad 7: /MOSI -> /GPIO3
- J5 pad 9: /MISO -> /SCK
Routing:
- net +3.3V: track 31.7 -> 59.4 mm, vias 3 -> 2
- net /SCL: track 0.00 -> 15.5 mm
- net /SDA: track 0.00 -> 14.6 mm
- net /MOSI: track 0.00 -> 14.0 mm
- net /MISO: track 0.00 -> 14.0 mm
- net /RESET: track 30.0 -> 16.1 mm
- net /SCK: track 0.00 -> 13.0 mm
- net /CS FRAM SPI: track 0.00 -> 12.2 mm
- net /CS BME280: track 0.00 -> 10.3 mm
- net /GPIO3: track 0.00 -> 9.44 mm
- net +5V: track 22.1 -> 29.3 mm

Commit message: zegar tesz
Parts:
- moved R5 9.97 mm to (186.0, 64.6), turned to 180 degrees
- moved C6 9.43 mm to (185.2, 51.9)
- moved SW2 9.43 mm to (179.2, 52.1)
- moved C5 8.60 mm to (185.1, 62.0)
- moved SW1 8.60 mm to (179.2, 62.0)
- moved C7 3.93 mm to (201.3, 60.4), turned to 180 degrees
- moved R4 2.76 mm to (186.9, 69.4), turned to -90 degrees
- moved R3 2.19 mm to (185.0, 69.4)
- moved C9 1.60 mm to (195.7, 60.6), turned to -90 degrees
- moved C10 0.39 mm to (198.7, 63.8)
- moved C11 0.28 mm to (207.6, 57.2)
- turned C4 to -90 degrees
Connections:
- J4 pad 10: /GPIO33 -> /MTDI
- J4 pad 12: /GPIO34 -> /MTDO
- J4 pad 14: /GPIO35 -> /MTCK
- J4 pad 16: /GPIO36 -> /GPIO38
- J4 pad 20: /GPIO38 -> /GPIO36
- J4 pad 22: /GPIO45 -> /GPIO35
- J4 pad 24: /GPIO46 -> /GPIO34
- J4 pad 3: /MTCK -> /XTAL_32K_P
- J4 pad 4: /MTDO -> /GPIO46
- J4 pad 5: /GPIO21 -> /XTAL_32K_N
- J4 pad 6: /MTDI -> /GPIO45
- J4 pad 7: /XTAL_32K_P -> /GPIO33
- J4 pad 9: /XTAL_32K_N -> /GPIO21
Routing:
- net +3.3V: track 59.4 -> 93.8 mm, vias 2 -> 5
- net /SCL: track 15.5 -> 46.6 mm
- net /SDA: track 14.6 -> 40.9 mm
- net /XTAL_32K_P: track 0.00 -> 23.2 mm, vias 0 -> 1
- net /GPIO34: track 0.00 -> 22.7 mm
- net /GPIO46: track 0.00 -> 22.2 mm
- net /GPIO45: track 0.00 -> 21.7 mm
- net /XTAL_32K_N: track 0.00 -> 21.3 mm, vias 0 -> 1
- net /GPIO35: track 0.00 -> 21.0 mm
- net /GPIO36: track 0.00 -> 20.1 mm
- net /GPIO37: track 0.00 -> 18.8 mm
- net /GPIO38: track 0.00 -> 18.5 mm
- net /GPIO21: track 0.00 -> 18.4 mm, vias 0 -> 1
- net /MTMS: track 0.00 -> 18.1 mm
- net /MTCK: track 0.00 -> 18.1 mm
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Other:
- board size 66.9 x 38.2 mm -> 55.9 x 38.2 mm
