File: Projekt_smiw.kicad_sch (KiCad schematic)
At the start: 25 parts, among them J1 USB_C_Receptacle_USB2.0, J2 Conn_01x08, J3 Conn_01x10, SW1 SW_Omron_B3FS, SW2 SW_Omron_B3FS, U1 USBLC6-2P6, U2 NCP1117-3.3_SOT223, U3 LM1117DT-3.3, U4 ESP32-S3-PICO-1

Commit message: wielka zmiena 2137
Connections:
- net CS BME280: now also J2.7 (Pin_7)
- net CS FRAM SPI: now also J2.8 (Pin_8); no longer J2.3 (Pin_3)
- net SCL: now also J2.3 (Pin_3); no longer J2.8 (Pin_8)
- net SDA: now also J2.2 (Pin_2); no longer J2.7 (Pin_7)
Changed lines of the file:
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@@
 	(wire
 		(pts
-			(xy 63.5 81.28) (xy 63.5 83.82)
+			(xy 140.97 139.7) (xy 143.51 139.7)
 		)
 		(stroke
@@
 	(wire
 		(pts
-			(xy 45.72 81.28) (xy 54.61 81.28)
+			(xy 63.5 81.28) (xy 63.5 83.82)
 		)
 		(stroke
@@
 	(wire
 		(pts
-			(xy 140.97 139.7) (xy 143.51 139.7)
+			(xy 45.72 81.28) (xy 54.61 81.28)
 		)
 		(stroke
@@
 	(wire
 		(pts
-			(xy 140.97 152.4) (xy 143.51 152.4)
+			(xy 45.72 76.2) (xy 54.61 76.2)
 		)
 		(stroke
@@
 	(wire
 		(pts
-			(xy 45.72 76.2) (xy 54.61 76.2)
+			(xy 189.23 86.36) (xy 193.04 86.36)
 		)
 		(stroke
@@
 	(wire
 		(pts
-			(xy 189.23 86.36) (xy 193.04 86.36)
+			(xy 140.97 149.86) (xy 143.51 149.86)
 		)
 		(stroke
@@
 	(wire
 		(pts
+			(xy 140.97 152.4) (xy 143.51 152.4)
+		)
+		(stroke
+			(width 0)
+			(type default)
+		)
+	)
+	(wire
+		(pts
 			(xy 125.73 69.85) (xy 125.73 72.39)
 		)
@@
 	(wire
 		(pts
-			(xy 179.07 50.8) (xy 176.53 50.8)
+			(xy 140.97 137.16) (xy 143.51 137.16)
 		)
 		(stroke
@@
 	(wire
 		(pts
-			(xy 140.97 149.86) (xy 143.51 149.86)
+			(xy 179.07 50.8) (xy 176.53 50.8)
 		)
 		(stroke
@@
 		)
 	)
-	(label "CS FRAM SPI"
-		(at 140.97 139.7 180)
+	(label "COL 3"
+		(at 158.75 139.7 0)
 		(effects
 			(font
 				(size 1.27 1.27)
 			)
-			(justify right bottom)
+			(justify left bottom)
 		)
 	)
-	(label "COL 3"
-		(at 158.75 139.7 0)
+	(label "SDA"
+		(at 140.97 137.16 180)
 		(effects
 			(font
 				(size 1.27 1.27)
 			)
-			(justify left bottom)
+			(justify right bottom)
 		)
 	)
@@
 		)
 	)
-	(label "SCL"
-		(at 140.97 152.4 180)
-		(effects
-			(font
-				(size 1.27 1.27)
-			)
-			(justify right bottom)
-		)
-	)
 	(label "COL 3"
 		(at 189.23 78.74 180)
@@
 		)
 	)
-	(label "SDA"
-		(at 140.97 149.86 180)
+	(label "CS FRAM SPI"
+		(at 140.97 152.4 180)
 		(effects
 			(font
@@
 		)
 	)
-	(label "CS BME280"
-		(at 140.97 137.16 180)
+	(label "SCL"
+		(at 140.97 139.7 180)
 		(effects
 			(font
@@
 		)
 	)
+	(label "CS BME280"
+		(at 140.97 149.86 180)
+		(effects
+			(font
+				(size 1.27 1.27)
+			)
+			(justify right bottom)
+		)
+	)
 	(symbol
 		(lib_id "power:GND")
@@
 			"0f20faa5-ef3f-4be0-bc53-31d21c09f398" "1146ef05-23e4-4aaa-afe9-edd3204370ef"
 			"18acbce2-de2f-43ee-92a6-d5121b3b753c" "1b792688-d4e0-405e-ab5f-70f2c2eb78f1"
-			"24f23426-a1c1-49f6-9db5-9e9787739f56" "26b79c05-79ca-498f-b28c-426acfac5fa8"
+			"1e11a7fa-a291-44dc-ac64-dfa8130ab6db" "26b79c05-79ca-498f-b28c-426acfac5fa8"
 			"2ac35770-718f-4a48-84e8-7df19a24203a" "3b690422-1398-4f19-a115-6a764ddf8ede"
 			"3fe701a3-8c52-498a-b8b6-cc78b9fede54" "41e67cd6-a75c-4af2-b0ce-c1721934d3a7"
-			"43c47642-6036-4ea5-967f-5fead81207b5" "4449d702-9a81-467e-9b27-92444aee10eb"
+			"4449d702-9a81-467e-9b27-92444aee10eb" "45d95596-47d2-4e7e-ad92-2d6045b1756f"
 			"4cd56b73-3206-410e-8566-ef1e8f544302" "4de851ac-7fe7-41a6-884b-0802e5a547a6"
 			"52148128-f05d-433c-aaa1-32bae2ef2238" "52c47359-2394-4bf0-a33c-6f364d16343a"
-			"586524f3-798c-4c2a-bdea-ce9d090938b2" "5e5daff2-0700-4f9c-9fe7-0c462b0a3ee9"
-			"6311a164-1a9f-46c7-b094-baa0c9354e04" "67d1b674-040a-4c28-9c4f-2dd3c573c629"
-			"7510b667-9784-44a3-9388-662601b5afc4" "7cd5e915-f442-4523-9c24-780c2e9336e1"
-			"89c14eaf-5962-47fe-8ab2-bbd188d53f35" "94c01670-2912-4f5c-a848-f296dd71f9aa"
+			"534ce8c5-fe9d-457d-a7ef-52eff13719e7" "586524f3-798c-4c2a-bdea-ce9d090938b2"
+			"5aaa75b8-2d07-464b-9517-997ea309081c" "67d1b674-040a-4c28-9c4f-2dd3c573c629"
+			"69cd27b2-b318-4a57-a143-c18f6577afc0" "7510b667-9784-44a3-9388-662601b5afc4"
+			"7cd5e915-f442-4523-9c24-780c2e9336e1" "89c14eaf-5962-47fe-8ab2-bbd188d53f35"
 			"9657c4ae-e888-4b50-8727-5b9f0c124c57" "9e721755-3b25-4e25-9e9e-5b7f326dde6b"
 			"b7078fb9-556c-42cd-9c72-1364b61bb7b2" "bed02eec-c0f3-402a-ba93-5a04d69a145a"
-			"c1f92fc0-29cd-4c20-afaa-2d7abac53f88" "c94cdee4-cb52-4543-aeeb-333f91e50149"
+			"c1f92fc0-29cd-4c20-afaa-2d7abac53f88" "caeb455f-2af0-49ea-9b7f-03a9cfb3c2a7"
 			"d0665d1e-2d99-400c-8d23-579234d2159c" "d5b7ff1f-5721-46bc-83dc-c01325e06c89"
-			"e0af1000-64cf-4d41-b3e3-b55613b95f97" "eab3a06f-78c8-40ab-9cbd-8287dd0071e0"
-			"f59b5e1a-80af-4df4-b6c4-3f88f4bdf7e3"
+			"e0af1000-64cf-4d41-b3e3-b55613b95f97" "eec5799f-8b9e-4203-8931-f29bff8c9659"
+			"f59b5e1a-80af-4df4-b6c4-3f88f4bdf7e3" "fc1aa054-aa18-42e8-86ad-55e3ecfba0a4"
 		)
 	)

Commit message: pvcv1
Parts:
- removed U3: LM1117DT-3.3, Package_TO_SOT_SMD:TO-252-3_TabPin2, symbol Regulator_Linear:LM1117DT-3.3
Connections:
- net SCL: now also J2.2 (Pin_2); no longer J2.3 (Pin_3)
- net SDA: now also J2.3 (Pin_3); no longer J2.2 (Pin_2)
Changed lines of the file:
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@@
 		)
 	)
-	(label "SDA"
+	(label "SCL"
 		(at 140.97 137.16 180)
 		(effects
@@
 		)
 	)
-	(label "SCL"
+	(label "SDA"
 		(at 140.97 139.7 180)
 		(effects
@@
 					(unit 1)
 				)
-			)
-		)
-	)
-	(symbol
-		(lib_id "Regulator_Linear:LM1117DT-3.3")
-		(at 77.47 60.96 0)
-		(unit 1)
-		(body_style 1)
-		(exclude_from_sim no)
-		(in_bom yes)
-		(on_board yes)
-		(in_pos_files yes)
-		(dnp no)
-		(fields_autoplaced yes)
-		(property "Reference" "U3"
-			(at 77.47 54.61 0)
-			(show_name no)
-			(do_not_autoplace no)
-			(effects
-				(font
-					(size 1.27 1.27)
-				)
-			)
-		)
-		(property "Value" "LM1117DT-3.3"
-			(at 77.47 57.15 0)
-			(show_name no)
-			(do_not_autoplace no)
-			(effects
-				(font
-					(size 1.27 1.27)
-				)
-			)
-		)
-		(property "Footprint" "Package_TO_SOT_SMD:TO-252-3_TabPin2"
-			(at 77.47 60.96 0)
-			(hide yes)
-			(show_name no)
-			(do_not_autoplace no)
-			(effects
-				(font
-					(size 1.27 1.27)
-				)
-			)
-		)
-		(property "Datasheet" "http://www.ti.com/lit/ds/symlink/lm1117.pdf"
-			(at 77.47 60.96 0)
-			(hide yes)
-			(show_name no)
-			(do_not_autoplace no)
-			(effects
-				(font
-					(size 1.27 1.27)
-				)
-			)
-		)
-		(property "Description" "800mA Low-Dropout Linear Regulator, 3.3V fixed output, TO-252"
-			(at 77.47 60.96 0)
-			(hide yes)
-			(show_name no)
-			(do_not_autoplace no)
-			(effects
-				(font
-					(size 1.27 1.27)
-				)
-			)
-		)
-		(pin "1"
-		)
-		(pin "2"
-		)
-		(pin "3"
-		)
-		(instances
-			(project "Projekt_smiw"
-				(path "/0969a27d-5e52-4b0c-8093-78bbacbcaa35"
-					(reference "U3")
-					(unit 1)
-				)

Commit message: Zmianakonnektora
Parts:
- removed J2: Conn_01x08, Connector_PinSocket_2.54mm:PinSocket_1x08_P2.54mm_Vertical, symbol Connector_Generic:Conn_01x08
- removed J3: Conn_01x10, Connector_PinSocket_2.54mm:PinSocket_1x10_P2.54mm_Vertical, symbol Connector_Generic:Conn_01x10
- added J4, J5: Conn_02x12_Odd_Even, symbol Connector_Generic:Conn_02x12_Odd_Even
Connections:
- net +3.3V: now also J4.1 (Pin_1), J4.3 (Pin_3), J5.1 (Pin_1), J5.2 (Pin_2)
- net COL 1: now also J5.4 (Pin_4)
- net COL 2: now also J5.6 (Pin_6)
- net COL 3: now also J5.8 (Pin_8)
- net COL 4: now also J5.10 (Pin_10)
- net CS BME280: now also J5.13 (Pin_13)
- net CS FRAM SPI: now also J5.15 (Pin_15)
- net GND: now also J4.15 (Pin_15), J4.17 (Pin_17), J4.19 (Pin_19), J4.21 (Pin_21), J4.23 (Pin_23), J5.19 (Pin_19), J5.20 (Pin_20), J5.21 (Pin_21), J5.22 (Pin_22), J5.23 (Pin_23), J5.24 (Pin_24)
- net MISO: now also J5.9 (Pin_9)
- net MOSI: now also J5.7 (Pin_7)
- net ROW 1: now also J5.12 (Pin_12)
- net ROW 2: now also J5.14 (Pin_14)
- net ROW 3: now also J5.16 (Pin_16)
- net ROW 4: now also J5.18 (Pin_18)
- net SCK: now also J5.11 (Pin_11)
- net SCL: now also J5.3 (Pin_3)
- net SDA: now also J5.5 (Pin_5)
- net XTAL_32K_P: now reaches U4.21 (XTAL_32K_P)
- net XTAL_32K_P: now also J4.7 (Pin_7)
- net XTAL_32K_N: now reaches U4.22 (XTAL_32K_N)
- net XTAL_32K_N: now also J4.9 (Pin_9)
- net GPIO21: now reaches U4.27 (GPIO21)
- net GPIO21: now also J4.5 (Pin_5)
- net SPICLK_N: now reaches U4.36 (SPICLK_N)
- net SPICLK_N: now also J4.13 (Pin_13)
- net SPICLK_P: now reaches U4.37 (SPICLK_P)
- net SPICLK_P: now also J4.11 (Pin_11)
- net GPIO33: now reaches U4.38 (GPIO33)
- net GPIO33: now also J4.10 (Pin_10)
- net GPIO34: now reaches U4.39 (GPIO34)
- net GPIO34: now also J4.12 (Pin_12)
- net GPIO35: now reaches U4.40 (GPIO35)
- net GPIO35: now also J4.14 (Pin_14)
- net GPIO36: now reaches U4.41 (GPIO36)
- net GPIO36: now also J4.16 (Pin_16)
- net GPIO37: now reaches U4.42 (GPIO37)
- net GPIO37: now also J4.18 (Pin_18)
- net GPIO38: now reaches U4.43 (GPIO38)
- net GPIO38: now also J4.20 (Pin_20)
- net MTCK: now reaches U4.44 (MTCK)
- net MTCK: now also J4.2 (Pin_2)
- net MTDO: now reaches U4.45 (MTDO)
- net MTDO: now also J4.4 (Pin_4)
- net MTDI: now reaches U4.47 (MTDI)
- net MTDI: now also J4.6 (Pin_6)
- net MTMS: now reaches U4.48 (MTMS)
- net MTMS: now also J4.8 (Pin_8)
- net UOTXD: now reaches U4.49 (U0TXD)
- net UORXD: now reaches U4.50 (U0RXD)
- net GPIO45: now reaches U4.51 (GPIO45)
- net GPIO45: now also J4.22 (Pin_22)
- net GPIO46: now reaches U4.52 (GPIO46)
- net GPIO46: now also J4.24 (Pin_24)
- net GPIO3: now reaches U4.8 (GPIO3)
- net GPIO3: now also J5.17 (Pin_17)
- no-connect marks 25 -> 5

Commit message: Zmianakonnektorav2
Parts:
- J4, J5: footprint (none) -> Connector_PinSocket_2.54mm:PinSocket_2x12_P2.54mm_Vertical
Connections:
- net +3.3V: now also J4.2 (Pin_2); no longer J4.3 (Pin_3)
- net MTCK: now also J4.3 (Pin_3); no longer J4.2 (Pin_2)
Changed lines of the file:
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@@
 	)
 	(junction
-		(at 251.46 133.35)
-		(diameter 0)
-		(color 0 0 0 0)
-	)
-	(junction
 		(at 251.46 153.67)
 		(diameter 0)
@@
 	(wire
 		(pts
+			(xy 269.24 132.08) (xy 269.24 133.35)
+		)
+		(stroke
+			(width 0)
+			(type default)
+		)
+	)
+	(wire
+		(pts
 			(xy 194.31 161.29) (xy 194.31 163.83)
 		)
@@
 	(wire
 		(pts
-			(xy 251.46 135.89) (xy 251.46 133.35)
-		)
-		(stroke
-			(width 0)
-			(type default)
-		)
-	)
-	(wire
-		(pts
 			(xy 63.5 44.45) (xy 77.47 44.45)
 		)
@@
 	(wire
 		(pts
+			(xy 269.24 133.35) (xy 266.7 133.35)
+		)
+		(stroke
+			(width 0)
+			(type default)
+		)
+	)
+	(wire
+		(pts
 			(xy 210.82 24.13) (xy 210.82 27.94)
 		)
@@
 	(wire
 		(pts
-			(xy 266.7 133.35) (xy 269.24 133.35)
-		)
-		(stroke
-			(width 0)
-			(type default)
-		)
-	)
-	(wire
-		(pts
 			(xy 218.44 48.26) (xy 218.44 49.53)
 		)
@@
 	)
 	(label "MTCK"
-		(at 269.24 133.35 0)
+		(at 251.46 135.89 180)
 		(effects
 			(font
 				(size 1.27 1.27)
 			)
-			(justify left bottom)
+			(justify right bottom)
 		)
 	)
@@
 			)
 		)
-		(property "Footprint" ""
+		(property "Footprint" "Connector_PinSocket_2.54mm:PinSocket_2x12_P2.54mm_Vertical"
 			(at 184.15 146.05 0)
 			(hide yes)
@@
 	)
 	(symbol
+		(lib_id "power:+3.3V")
+		(at 269.24 132.08 0)
+		(unit 1)
+		(body_style 1)
+		(exclude_from_sim no)
+		(in_bom yes)
+		(on_board yes)
+		(in_pos_files yes)
+		(dnp no)
+		(fields_autoplaced yes)
+		(property "Reference" "#PWR024"
+			(at 269.24 135.89 0)
+			(hide yes)
+			(show_name no)
+			(do_not_autoplace no)
+			(effects
+				(font
+					(size 1.27 1.27)
+				)
+			)
+		)
+		(property "Value" "+3.3V"
+			(at 269.24 127 0)
+			(show_name no)
+			(do_not_autoplace no)
+			(effects
+				(font
+					(size 1.27 1.27)
+				)
+			)
+		)
+		(property "Footprint" ""
+			(at 269.24 132.08 0)
+			(hide yes)
+			(show_name no)
+			(do_not_autoplace no)
+			(effects
+				(font
+					(size 1.27 1.27)
+				)
+			)
+		)
+		(property "Datasheet" ""
+			(at 269.24 132.08 0)
+			(hide yes)
+			(show_name no)
+			(do_not_autoplace no)
+			(effects
+				(font
+					(size 1.27 1.27)
+				)
+			)
+		)
+		(property "Description" "Power symbol creates a global label with name \"+3.3V\""
+			(at 269.24 132.08 0)
+			(hide yes)
+			(show_name no)
+			(do_not_autoplace no)
+			(effects
+				(font
+					(size 1.27 1.27)
+				)
+			)
+		)
+		(pin "1"
+		)
+		(instances
+			(project "Projekt_smiw"
+				(path "/0969a27d-5e52-4b0c-8093-78bbacbcaa35"
+					(reference "#PWR024")
+					(unit 1)
+				)
+			)
+		)
+	)
+	(symbol
 		(lib_id "power:GND")
 		(at 125.73 72.39 0)
@@
 			)
 		)
-		(property "Footprint" ""
+		(property "Footprint" "Connector_PinSocket_2.54mm:PinSocket_2x12_P2.54mm_Vertical"
 			(at 259.08 146.05 0)
 			(hide yes)

Commit message: poprawkaconnector
Connections:
- net CS BME280: now also J5.5 (Pin_5); no longer J5.13 (Pin_13)
- net CS FRAM SPI: now also J5.3 (Pin_3); no longer J5.15 (Pin_15)
- net GPIO3: now also J5.7 (Pin_7); no longer J5.17 (Pin_17)
- net MISO: now also J5.11 (Pin_11); no longer J5.9 (Pin_9)
- net MOSI: now also J5.13 (Pin_13); no longer J5.7 (Pin_7)
- net SCK: now also J5.9 (Pin_9); no longer J5.11 (Pin_11)
- net SCL: now also J5.17 (Pin_17); no longer J5.3 (Pin_3)
- net SDA: now also J5.15 (Pin_15); no longer J5.5 (Pin_5)
Changed lines of the file:
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@@
 	)
 	(label "SCK"
-		(at 176.53 146.05 180)
+		(at 176.53 143.51 180)
 		(effects
 			(font
@@
 	)
 	(label "SDA"
-		(at 176.53 138.43 180)
+		(at 176.53 151.13 180)
 		(effects
 			(font
@@
 	)
 	(label "MISO"
-		(at 176.53 143.51 180)
+		(at 176.53 146.05 180)
 		(effects
 			(font
@@
 	)
 	(label "CS FRAM SPI"
-		(at 176.53 151.13 180)
+		(at 176.53 135.89 180)
 		(effects
 			(font
@@
 	)
 	(label "SCL"
-		(at 176.53 135.89 180)
+		(at 176.53 153.67 180)
 		(effects
 			(font
@@
 	)
 	(label "CS BME280"
-		(at 176.53 148.59 180)
+		(at 176.53 138.43 180)
 		(effects
 			(font
@@
 	)
 	(label "GPIO3"
-		(at 176.53 153.67 180)
+		(at 176.53 140.97 180)
 		(effects
 			(font
@@
 	)
 	(label "MOSI"
-		(at 176.53 140.97 180)
-		(effects
-			(font
+		(at 176.53 148.59 180)
+		(effects
+			(font

Commit message: zegar tesz
Connections:
- net GPIO21: now also J4.9 (Pin_9); no longer J4.5 (Pin_5)
- net GPIO33: now also J4.7 (Pin_7); no longer J4.10 (Pin_10)
- net GPIO34: now also J4.24 (Pin_24); no longer J4.12 (Pin_12)
- net GPIO35: now also J4.22 (Pin_22); no longer J4.14 (Pin_14)
- net GPIO36: now also J4.20 (Pin_20); no longer J4.16 (Pin_16)
- net GPIO38: now also J4.16 (Pin_16); no longer J4.20 (Pin_20)
- net GPIO45: now also J4.6 (Pin_6); no longer J4.22 (Pin_22)
- net GPIO46: now also J4.4 (Pin_4); no longer J4.24 (Pin_24)
- net MTCK: now also J4.14 (Pin_14); no longer J4.3 (Pin_3)
- net MTDI: now also J4.10 (Pin_10); no longer J4.6 (Pin_6)
- net MTDO: now also J4.12 (Pin_12); no longer J4.4 (Pin_4)
- net XTAL_32K_N: now also J4.5 (Pin_5); no longer J4.9 (Pin_9)
- net XTAL_32K_P: now also J4.3 (Pin_3); no longer J4.7 (Pin_7)
Changed lines of the file:
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@@
+	(wire
+		(pts
+			(xy 266.7 158.75) (xy 269.24 158.75)
+		)
+		(stroke
+			(width 0)
+			(type default)
+		)
+	)
 	(wire
 		(pts
@@
 	(wire
 		(pts
-			(xy 254 135.89) (xy 251.46 135.89)
-		)
-		(stroke
-			(width 0)
-			(type default)
-		)
-	)
-	(wire
-		(pts
 			(xy 251.46 158.75) (xy 254 158.75)
 		)
@@
 	(wire
 		(pts
+			(xy 251.46 135.89) (xy 254 135.89)
+		)
+		(stroke
+			(width 0)
+			(type default)
+		)
+	)
+	(wire
+		(pts
 			(xy 215.9 40.64) (xy 215.9 49.53)
 		)
@@
 	(wire
 		(pts
+			(xy 266.7 148.59) (xy 269.24 148.59)
+		)
+		(stroke
+			(width 0)
+			(type default)
+		)
+	)
+	(wire
+		(pts
 			(xy 266.7 138.43) (xy 269.24 138.43)
 		)
@@
 	(wire
 		(pts
-			(xy 266.7 158.75) (xy 269.24 158.75)
-		)
-		(stroke
-			(width 0)
-			(type default)
-		)
-	)
-	(wire
-		(pts
 			(xy 72.39 68.58) (xy 72.39 73.66)
 		)
@@
 		(pts
 			(xy 251.46 153.67) (xy 254 153.67)
-		)
-		(stroke
-			(width 0)
-			(type default)
-		)
-	)
-	(wire
-		(pts
-			(xy 266.7 148.59) (xy 269.24 148.59)
 		)
 		(stroke
@@
 	)
 	(label "GPIO46"
-		(at 269.24 161.29 0)
+		(at 269.24 135.89 0)
 		(effects
 			(font
@@
 	)
 	(label "GPIO36"
-		(at 269.24 151.13 0)
+		(at 269.24 156.21 0)
 		(effects
 			(font
@@
 	)
 	(label "GPIO33"
-		(at 269.24 143.51 0)
-		(effects
-			(font
-				(size 1.27 1.27)
-			)
-			(justify left bottom)
+		(at 251.46 140.97 180)
+		(effects
+			(font
+				(size 1.27 1.27)
+			)
+			(justify right bottom)
 		)
 	)
@@
 	)
 	(label "MTCK"
-		(at 251.46 135.89 180)
-		(effects
-			(font
-				(size 1.27 1.27)
-			)
-			(justify right bottom)
+		(at 269.24 148.59 0)
+		(effects
+			(font
+				(size 1.27 1.27)
+			)
+			(justify left bottom)
 		)
 	)
@@
 	)
 	(label "GPIO34"
-		(at 269.24 146.05 0)
+		(at 269.24 161.29 0)
 		(effects
 			(font
@@
 	)
 	(label "GPIO21"
-		(at 251.46 138.43 180)
+		(at 251.46 143.51 180)
 		(effects
 			(font
@@
 	)
 	(label "MTDO"
-		(at 269.24 135.89 0)
+		(at 269.24 146.05 0)
 		(effects
 			(font
@@
 	)
 	(label "GPIO45"
-		(at 269.24 158.75 0)
+		(at 269.24 138.43 0)
 		(effects
 			(font
@@
 	)
 	(label "GPIO38"
-		(at 269.24 156.21 0)
+		(at 269.24 151.13 0)
 		(effects
 			(font
@@
 	)
 	(label "XTAL_32K_N"
-		(at 251.46 143.51 180)
+		(at 251.46 138.43 180)
 		(effects
 			(font
@@
 	)
 	(label "MTDI"
-		(at 269.24 138.43 0)
+		(at 269.24 143.51 0)
 		(effects
 			(font
@@
 	)
 	(label "GPIO35"
-		(at 269.24 148.59 0)
+		(at 269.24 158.75 0)
 		(effects
 			(font
@@
 	)
 	(label "XTAL_32K_P"
-		(at 251.46 140.97 180)
-		(effects
-			(font
+		(at 251.46 135.89 180)
+		(effects
+			(font
