File: klawiaturka/klawiaturka.kicad_sch (KiCad schematic)
At the start: 22 parts, among them J6 Conn_01x08, J7 Conn_01x10, SW10 SW_Push, SW11 SW_Push, SW12 SW_Push, SW13 SW_Push, SW14 SW_Push, SW15 SW_Push, SW16 SW_Push, SW17 SW_Push, SW18 SW_Push, SW3 SW_Push, SW4 SW_Push, SW5 SW_Push, SW6 SW_Push, SW7 SW_Push, SW8 SW_Push, SW9 SW_Push

Commit message: :3 x2
Parts:
- renumbered SW3 to SW1
Connections:
- net CS BME280: now also J6.7 (Pin_7); no longer J6.2 (Pin_2)
- net CS FRAM SPI: now also J6.8 (Pin_8); no longer J6.3 (Pin_3)
- net SCL: now also J6.2 (Pin_2); no longer J6.8 (Pin_8)
- net SDA: now also J6.3 (Pin_3); no longer J6.7 (Pin_7)
Changed lines of the file:
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@@
 	(wire
 		(pts
-			(xy 194.31 71.12) (xy 196.85 71.12)
+			(xy 99.06 116.84) (xy 99.06 120.65)
 		)
 		(stroke
@@
 	(wire
 		(pts
-			(xy 99.06 116.84) (xy 99.06 120.65)
+			(xy 78.74 116.84) (xy 80.01 116.84)
 		)
 		(stroke
@@
 	(wire
 		(pts
-			(xy 78.74 116.84) (xy 80.01 116.84)
+			(xy 119.38 151.13) (xy 140.97 151.13)
 		)
 		(stroke
@@
 	(wire
 		(pts
-			(xy 119.38 151.13) (xy 140.97 151.13)
+			(xy 194.31 68.58) (xy 196.85 68.58)
 		)
 		(stroke
@@
 	(wire
 		(pts
+			(xy 194.31 55.88) (xy 196.85 55.88)
+		)
+		(stroke
+			(width 0)
+			(type default)
+		)
+	)
+	(wire
+		(pts
 			(xy 99.06 101.6) (xy 99.06 105.41)
 		)
@@
 	(wire
 		(pts
-			(xy 194.31 58.42) (xy 196.85 58.42)
+			(xy 194.31 71.12) (xy 196.85 71.12)
 		)
 		(stroke
@@
 	(wire
 		(pts
+			(xy 194.31 58.42) (xy 196.85 58.42)
+		)
+		(stroke
+			(width 0)
+			(type default)
+		)
+	)
+	(wire
+		(pts
 			(xy 74.93 120.65) (xy 78.74 120.65)
 		)
@@
 	(wire
 		(pts
-			(xy 194.31 55.88) (xy 196.85 55.88)
-		)
-		(stroke
-			(width 0)
-			(type default)
-		)
-	)
-	(wire
-		(pts
 			(xy 113.03 76.2) (xy 113.03 80.01)
 		)
@@
 	(wire
 		(pts
-			(xy 194.31 68.58) (xy 196.85 68.58)
-		)
-		(stroke
-			(width 0)
-			(type default)
-		)
-	)
-	(wire
-		(pts
 			(xy 153.67 132.08) (xy 153.67 147.32)
 		)
@@
 		)
 	)
+	(label "SCL"
+		(at 194.31 55.88 180)
+		(effects
+			(font
+				(size 1.27 1.27)
+			)
+			(justify right bottom)
+		)
+	)
 	(label "SCK"
 		(at 194.31 66.04 180)
@@
 		)
 	)
-	(label "CS BME280"
-		(at 194.31 55.88 180)
-		(effects
-			(font
-				(size 1.27 1.27)
-			)
-			(justify right bottom)
-		)
-	)
 	(label "ROW 1"
 		(at 212.09 63.5 0)
@@
 		)
 	)
-	(label "SDA"
+	(label "CS BME280"
 		(at 194.31 68.58 180)
 		(effects
@@
 	)
 	(label "CS FRAM SPI"
+		(at 194.31 71.12 180)
+		(effects
+			(font
+				(size 1.27 1.27)
+			)
+			(justify right bottom)
+		)
+	)
+	(label "SDA"
 		(at 194.31 58.42 180)
 		(effects
@@
 		)
 	)
-	(label "SCL"
-		(at 194.31 71.12 180)
-		(effects
-			(font
-				(size 1.27 1.27)
-			)
-			(justify right bottom)
-		)
-	)
 	(label "COL 3"
 		(at 133.35 76.2 0)
@@
 				)
 			)
+			(project "klawiaturka"
+				(path "/6f31acde-a091-40b7-8cc4-b5bb83c555ef"
+					(reference "SW12")
+					(unit 1)
+				)
+			)
 		)
 	)
@@
 				)
 			)
+			(project "klawiaturka"
+				(path "/6f31acde-a091-40b7-8cc4-b5bb83c555ef"
+					(reference "SW8")
+					(unit 1)
+				)
+			)
 		)
 	)
@@
 				)
 			)
+			(project "klawiaturka"
+				(path "/6f31acde-a091-40b7-8cc4-b5bb83c555ef"
+					(reference "SW11")
+					(unit 1)
+				)
+			)
 		)
 	)
@@
 				)
 			)
+			(project "klawiaturka"
+				(path "/6f31acde-a091-40b7-8cc4-b5bb83c555ef"
+					(reference "SW15")
+					(unit 1)
+				)
+			)
 		)
 	)
@@
 				)
 			)
+			(project "klawiaturka"
+				(path "/6f31acde-a091-40b7-8cc4-b5bb83c555ef"
+					(reference "SW6")
+					(unit 1)
+				)
+			)
 		)
 	)
@@
 		(dnp no)
 		(fields_autoplaced yes)
-		(property "Reference" "SW3"
+		(property "Reference" "SW1"
 			(at 85.09 93.98 0)
 			(show_name no)
@@
 				)
 			)
+			(project "klawiaturka"
+				(path "/6f31acde-a091-40b7-8cc4-b5bb83c555ef"
+					(reference "SW9")
+					(unit 1)
+				)
+			)
 		)
 	)
@@
 				)
 			)
+			(project "klawiaturka"
+				(path "/6f31acde-a091-40b7-8cc4-b5bb83c555ef"
+					(reference "SW16")
+					(unit 1)
+				)
+			)
 		)
 	)
@@
 				)
 			)
+			(project "klawiaturka"
+				(path "/6f31acde-a091-40b7-8cc4-b5bb83c555ef"
+					(reference "SW5")
+					(unit 1)
+				)
+			)
 		)
 	)
@@
 				)
 			)
+			(project "klawiaturka"
+				(path "/6f31acde-a091-40b7-8cc4-b5bb83c555ef"
+					(reference "#PWR029")
+					(unit 1)
+				)
+			)
 		)
 	)
@@
 				)
 			)
+			(project "klawiaturka"
+				(path "/6f31acde-a091-40b7-8cc4-b5bb83c555ef"
+					(reference "SW4")
+					(unit 1)
+				)
+			)
 		)
 	)
@@
 				)
 			)
+			(project "klawiaturka"
+				(path "/6f31acde-a091-40b7-8cc4-b5bb83c555ef"
+					(reference "SW13")
+					(unit 1)
+				)
+			)
 		)
 	)
@@
 				)
 			)
+			(project "klawiaturka"
+				(path "/6f31acde-a091-40b7-8cc4-b5bb83c555ef"
+					(reference "SW7")
+					(unit 1)
+				)
+			)
 		)
 	)
@@
 				)
 			)
+			(project "klawiaturka"
+				(path "/6f31acde-a091-40b7-8cc4-b5bb83c555ef"
+					(reference "SW10")
+					(unit 1)
+				)
+			)
 		)
 	)
@@
 				)
 			)
+			(project "klawiaturka"
+				(path "/6f31acde-a091-40b7-8cc4-b5bb83c555ef"
+					(reference "SW14")
+					(unit 1)
+				)
+			)
 		)
 	)
@@
 				)
 			)
+			(project "klawiaturka"
+				(path "/6f31acde-a091-40b7-8cc4-b5bb83c555ef"
+					(reference "SW17")
+					(unit 1)
+				)
+			)
 		)
 	)
@@
 				)
 			)
+			(project "klawiaturka"
+				(path "/6f31acde-a091-40b7-8cc4-b5bb83c555ef"
+					(reference "J6")
+					(unit 1)
+				)
+			)
 		)
 	)
@@
 				)
 			)
+			(project "klawiaturka"
+				(path "/6f31acde-a091-40b7-8cc4-b5bb83c555ef"
+					(reference "J7")
+					(unit 1)
+				)
+			)
 		)
 	)
@@
 				)
 			)
+			(project "klawiaturka"
+				(path "/6f31acde-a091-40b7-8cc4-b5bb83c555ef"
+					(reference "#PWR030")
+					(unit 1)
+				)
+			)
 		)
 	)
@@
 				)
 			)
+			(project "klawiaturka"
+				(path "/6f31acde-a091-40b7-8cc4-b5bb83c555ef"
+					(reference "SW18")
+					(unit 1)
+				)
+			)
 		)
 	)
 	(group "conn"
 		(members "045f02d7-7aa9-47ce-9b71-affe68a4c37e" "1bdacc7d-cf53-4979-bd4a-ef14e8e1f974"
-			"1d38e008-4c74-48fb-91fd-ab4876f88a21" "1f7097bc-6ead-4548-9657-2002ead8e0b0"
-			"2a7107ae-8c48-49d8-87ff-78652665cb5d" "3332caad-0a42-4220-8f77-73e6af7a04db"
-			"34eabbb3-5d22-48b7-9fde-60d14454d91f" "38ba6e10-7bcf-498f-90e8-09f073948d79"
-			"4aa7dcc3-85df-4891-8b95-7bad9d0cae5f" "53fff72f-7494-4200-a7b7-7e486365f5c5"
+			"1f7097bc-6ead-4548-9657-2002ead8e0b0" "21825de0-8377-4f26-b1ab-0adb2a7454fe"
+			"2a7107ae-8c48-49d8-87ff-78652665cb5d" "2f54035a-2f31-4c88-b8a6-b18ab0806e7c"
+			"3332caad-0a42-4220-8f77-73e6af7a04db" "34eabbb3-5d22-48b7-9fde-60d14454d91f"
+			"38ba6e10-7bcf-498f-90e8-09f073948d79" "4aa7dcc3-85df-4891-8b95-7bad9d0cae5f"
+			"4b2555b4-7e5f-4749-b105-fc61f43310bc" "57499524-363a-4e54-b88f-9c6f05b09fa2"
 			"5f4f50d2-fba3-4d71-97ce-80529ead0c3f" "66b8eacd-c592-4050-8236-553c545aa362"
 			"69d168ae-dfb8-49b0-b66a-57ec6532c545" "6f8683a5-9f74-4c22-9d3a-dde37785d7d4"
-			"79051540-9062-4276-a92b-97a1bb563576" "84885a11-8552-4e2a-81ff-43cae9fccd26"
-			"8fccb2cc-946f-4c6f-8382-601f25c06cb3" "901467d7-e2ab-401c-9f80-03081a7a710b"
-			"9043ee0a-00d7-4bcf-af12-a07864cf8647" "933d73a0-44a6-4b81-a066-f8888f89b217"
-			"97e9df2d-143d-4231-957f-a2ae933f75f7" "9c6a93e4-1f70-4940-aa0b-03bd899f7405"
-			"9e1f0542-5a95-4d42-a759-be56d059a258" "9f907049-deed-4f5b-b7dd-2f155df1de2e"
-			"a3ff899f-a157-4c14-b7b4-08b02204731a" "af9f6d3f-116d-4059-a742-1e3fb6f5b976"
-			"b0cce12e-7cb0-4b97-94b4-58ee79e0ff09" "b2fbd65c-c850-4228-bcd9-15bdddb08306"
-			"c4a12e6e-4ac6-49e2-8973-442fa4eae3ec" "cf4d2e00-2afa-46df-80b6-826f04499636"
+			"73dcecfe-f886-4866-b511-4e6f857182e7" "79051540-9062-4276-a92b-97a1bb563576"
+			"84885a11-8552-4e2a-81ff-43cae9fccd26" "8fccb2cc-946f-4c6f-8382-601f25c06cb3"
+			"901467d7-e2ab-401c-9f80-03081a7a710b" "933d73a0-44a6-4b81-a066-f8888f89b217"
+			"9c6a93e4-1f70-4940-aa0b-03bd899f7405" "9f907049-deed-4f5b-b7dd-2f155df1de2e"
+			"a3ff899f-a157-4c14-b7b4-08b02204731a" "a4318a2c-d058-4f06-83dc-b1a4e91514b2"
+			"af9f6d3f-116d-4059-a742-1e3fb6f5b976" "b0cce12e-7cb0-4b97-94b4-58ee79e0ff09"
+			"b2fbd65c-c850-4228-bcd9-15bdddb08306" "bcd5afb9-8891-4cd9-9b17-4499cb4d5b3d"
+			"becf5c97-f4fc-4d28-a809-7aa3e46a4a1e" "cf4d2e00-2afa-46df-80b6-826f04499636"
 			"d0a84248-a443-4f90-983e-92b822c1e6b1" "d3c22ba0-3059-4a39-baa5-7008bee10aa4"
 			"d5ed38b6-6b40-41e3-a7ff-1f378759a3a7" "d64d1c85-ddcf-4698-ab64-bd4f4ef04966"
 			"e11c312a-fc22-4b83-a01a-2219b4f0bdcc" "e25a6f0c-bc17-411d-81a1-f693891c7bc4"
-			"e70267b8-25e3-40c4-8580-5aad82e5174c" "f877325c-6844-4ee5-859f-8681b0b641fc"
-			"f8e1d27b-0d3e-488b-8b50-9e3e8f4e8f1e" "fe60c96d-2804-43cb-ac01-82608b86486c"
+			"f877325c-6844-4ee5-859f-8681b0b641fc" "fe60c96d-2804-43cb-ac01-82608b86486c"
 		)
 	)
@@
 		)
 	)
+	(embedded_fonts no)
 )

Commit message: Zmianakonnektora
Parts:
- removed J6: Conn_01x08, Connector_PinHeader_2.54mm:PinHeader_1x08_P2.54mm_Vertical, symbol Connector_Generic:Conn_01x08
- removed J7: Conn_01x10, Connector_PinHeader_2.54mm:PinHeader_1x10_P2.54mm_Vertical, symbol Connector_Generic:Conn_01x10
- added J4, J5: Conn_02x12_Odd_Even, Connector_PinSocket_2.54mm:PinSocket_2x12_P2.54mm_Vertical, symbol Connector_Generic:Conn_02x12_Odd_Even
Connections:
- net +3.3V: now also J4.1 (Pin_1), J4.3 (Pin_3), J5.1 (Pin_1), J5.2 (Pin_2)
- net COL 1: now also J5.4 (Pin_4)
- net COL 2: now also J5.6 (Pin_6)
- net COL 3: now also J5.8 (Pin_8)
- net COL 4: now also J5.10 (Pin_10)
- net CS BME280: now also J5.13 (Pin_13)
- net CS FRAM SPI: now also J5.15 (Pin_15)
- net GND: now also J4.15 (Pin_15), J4.17 (Pin_17), J4.19 (Pin_19), J4.21 (Pin_21), J4.23 (Pin_23), J5.19 (Pin_19), J5.20 (Pin_20), J5.21 (Pin_21), J5.22 (Pin_22), J5.23 (Pin_23), J5.24 (Pin_24)
- net MISO: now also J5.9 (Pin_9)
- net MOSI: now also J5.7 (Pin_7)
- net ROW 1: now also J5.12 (Pin_12)
- net ROW 2: now also J5.14 (Pin_14)
- net ROW 3: now also J5.16 (Pin_16)
- net ROW 4: now also J5.18 (Pin_18)
- net SCK: now also J5.11 (Pin_11)
- net SCL: now also J5.3 (Pin_3)
- net SDA: now also J5.5 (Pin_5)
- new net GPIO21: J4.5 (Pin_5)
- new net GPIO3: J5.17 (Pin_17)
- new net GPIO33: J4.10 (Pin_10)
- new net GPIO34: J4.12 (Pin_12)
- new net GPIO35: J4.14 (Pin_14)
- new net GPIO36: J4.16 (Pin_16)
- new net GPIO37: J4.18 (Pin_18)
- new net GPIO38: J4.20 (Pin_20)
- new net GPIO45: J4.22 (Pin_22)
- new net GPIO46: J4.24 (Pin_24)
- new net MTCK: J4.2 (Pin_2)
- new net MTDI: J4.6 (Pin_6)
- new net MTDO: J4.4 (Pin_4)
- new net MTMS: J4.8 (Pin_8)
- new net SPICLK_N: J4.13 (Pin_13)
- new net SPICLK_P: J4.11 (Pin_11)
- new net XTAL_32K_N: J4.9 (Pin_9)
- new net XTAL_32K_P: J4.7 (Pin_7)

Commit message: Zmianakonnektorav2
Connections:
- net +3.3V: now also J4.2 (Pin_2); no longer J4.3 (Pin_3)
- net MTCK: now also J4.3 (Pin_3); no longer J4.2 (Pin_2)
