File: klawiaturka/klawiaturka.kicad_pcb (KiCad board)
At the start: 2 copper layers, 22 parts, among them J6 Conn_01x08, J7 Conn_01x10, SW1 SW_Push, SW10 SW_Push, SW11 SW_Push, SW12 SW_Push, SW13 SW_Push, SW14 SW_Push, SW15 SW_Push, SW16 SW_Push, SW17 SW_Push, SW18 SW_Push, SW4 SW_Push, SW5 SW_Push, SW6 SW_Push, SW7 SW_Push, SW8 SW_Push, SW9 SW_Push

Commit message: Płytka PCB z klawiaturki v1
Parts:
- moved J7 106.3 mm to (76.0, 85.2)
- moved D1 86.2 mm to (101.0, 73.3), turned to -90 degrees
- moved D2 66.5 mm to (121.5, 72.7), turned to -90 degrees
- moved D3 46.0 mm to (143.5, 72.7), turned to -90 degrees
- moved SW3 42.7 mm to (93.5, 83.8)
- moved SW4 42.7 mm to (93.5, 91.7)
- moved SW5 42.7 mm to (93.5, 99.5)
- moved SW6 42.7 mm to (93.5, 107.3)
- moved SW10 33.0 mm to (114.5, 107.0)
- moved SW7 33.0 mm to (114.5, 83.5)
- moved SW8 33.0 mm to (114.5, 91.3)
- moved SW9 33.0 mm to (114.5, 99.2)
- moved D4 27.5 mm to (166.0, 73.0), turned to -90 degrees
- moved SW11 23.8 mm to (135.0, 83.5)
- moved SW12 23.8 mm to (135.0, 91.3)
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- renumbered SW1 to SW3
Routing:
- net /ROW 1: track 0.00 -> 242.3 mm, vias 0 -> 3
- net /ROW 2: track 0.00 -> 226.1 mm, vias 0 -> 3
- net /ROW 3: track 0.00 -> 201.5 mm, vias 0 -> 3
- net /ROW 4: track 0.00 -> 177.1 mm, vias 0 -> 3
- net /COL 4: track 0.00 -> 99.8 mm, vias 0 -> 1
- net Net-(D4-A): track 0.00 -> 90.7 mm
- net Net-(D3-A): track 0.00 -> 88.8 mm
- net Net-(D1-A): track 0.00 -> 83.8 mm
- net /COL 3: track 0.00 -> 82.2 mm, vias 0 -> 1
- net Net-(D2-A): track 0.00 -> 81.8 mm
- net /COL 2: track 0.00 -> 57.9 mm, vias 0 -> 1
- net /COL 1: track 0.00 -> 32.0 mm, vias 0 -> 1
- net GND: track 0.00 -> 2.54 mm
Other:
- board outline added: 98.5 x 49 mm
- copper layers 2 -> 4

Commit message: KlawiaturkaV2
Parts:
- removed J6: Conn_01x08, Connector_PinHeader_2.54mm:PinHeader_1x08_P2.54mm_Vertical
- removed J7: Conn_01x10, Connector_PinHeader_2.54mm:PinHeader_1x10_P2.54mm_Vertical
- added J4: Conn_02x12_Odd_Even, Connector_PinSocket_2.54mm:PinSocket_2x12_P2.54mm_Vertical, F.Cu at (221.9, 34.8)
- added J5: Conn_02x12_Odd_Even, Connector_PinSocket_2.54mm:PinSocket_2x12_P2.54mm_Vertical, F.Cu at (221.9, 62.8)
- moved D1 96.7 mm to (197.7, 74.6)
- moved SW4 95.5 mm to (188.7, 84.3)
- moved SW3 95.5 mm to (188.7, 76.5)
- moved SW5 95.5 mm to (188.7, 92.2)
- moved SW6 95.5 mm to (188.7, 100.0)
- moved D2 93.8 mm to (215.3, 74.6)
- moved SW10 92.1 mm to (206.3, 100.0)
- moved SW7 92.1 mm to (206.3, 76.5)
- moved SW8 92.1 mm to (206.3, 84.3)
- moved SW9 92.1 mm to (206.3, 92.2)
- moved SW11 89.2 mm to (223.9, 76.5)
- moved SW12 89.2 mm to (223.9, 84.3)
- moved SW13 89.2 mm to (223.9, 92.2)
- moved SW14 89.2 mm to (223.9, 100.0)
- moved D3 88.4 mm to (231.9, 74.6)
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Routing:
- net /ROW 1: track 242.3 -> 132.8 mm, vias 3 -> 4
- net /COL 4: track 99.8 -> 9.52 mm, vias 1 -> 0
- net /ROW 2: track 226.1 -> 144.3 mm, vias 3 -> 4
- net /COL 3: track 82.2 -> 9.48 mm, vias 1 -> 0
- net /ROW 3: track 201.5 -> 152.0 mm, vias 3 -> 4
- net /COL 2: track 57.9 -> 15.2 mm, vias 1 -> 0
- net Net-(D4-A): track 90.7 -> 71.5 mm
- net Net-(D3-A): track 88.8 -> 75.2 mm
- net /ROW 4: track 177.1 -> 166.9 mm, vias 3 -> 4
- net GND: track 2.54 -> 0.00 mm
- net Net-(D1-A): track 83.8 -> 81.5 mm
- net Net-(D2-A): track 81.8 -> 79.6 mm
- net /COL 1: track 32.0 -> 30.2 mm, vias 1 -> 0
Other:
- board size 98.5 x 49 mm -> 71.8 x 75 mm
