File: czujnik/czujnik.kicad_pcb (KiCad board)
At the start: 2 copper layers, 9 parts, among them J4 Conn_01x08, J5 Conn_01x10, U5 BME280, U6 MB85RS256B

Commit message: awetg2
Parts:
- moved R7 91.8 mm to (102.4, 128.5), turned to 0 degrees
- moved J5 88.1 mm to (102.5, 136.9), turned to 90 degrees
- moved C13 86.0 mm to (108.8, 121.7), turned to 0 degrees
- moved R6 86.0 mm to (103.5, 121.0), turned to 0 degrees
- moved C12 79.1 mm to (111.5, 100.8)
- moved C14 79.1 mm to (110.8, 103.3)
- moved U5 79.1 mm to (114.5, 103.3)
- moved U6 78.9 mm to (113.0, 126.5), turned to 90 degrees
- moved J4 60.3 mm to (125.4, 115.1)
Routing:
- net +3.3V: track 0.00 -> 3.56 mm
- removed copper zone on B.Cu, net GND
Other:
- copper layers 2 -> 4

Commit message: czujnik pcb
Parts:
- R7: moved to B.Cu
- moved R6 9.76 mm to (112.4, 117.0), turned to -90 degrees
- moved C14 8.96 mm to (112.3, 112.1), turned to 90 degrees
- moved R7 8.94 mm to (110.8, 131.7)
- moved C12 7.56 mm to (112.3, 108.3)
- moved U5 7.07 mm to (115.0, 110.3)
Connections:
- J4 pad 2: /CS BME280 -> /SCL
- J4 pad 3: /CS FRAM SPI -> /SDA
- J4 pad 7: /SDA -> /CS BME280
- J4 pad 8: /SCL -> /CS FRAM SPI
Routing:
- net +3.3V: track 3.56 -> 54.2 mm, vias 0 -> 1
- net /MISO: track 0.00 -> 38.7 mm, vias 0 -> 1
- net /SCK: track 0.00 -> 29.9 mm, vias 0 -> 2
- net /MOSI: track 0.00 -> 27.1 mm, vias 0 -> 2
- net /CS BME280: track 0.00 -> 25.8 mm, vias 0 -> 1
- net /CS FRAM SPI: track 0.00 -> 16.5 mm
- net Net-(U6-~{HOLD}): track 0.00 -> 6.84 mm
- net Net-(U6-~{WP}): track 0.00 -> 6.00 mm, vias 0 -> 1
- added copper zone on B.Cu, net GND
- added copper zone on F.Cu, net GND

Commit message: :3
Routing:
- net /MOSI: track 27.1 -> 30.2 mm, vias 2 -> 1
- net GND: track 0.00 -> 0.75 mm, vias 0 -> 1
- net /MISO: track 38.7 -> 39.4 mm
Other:
- board outline added: 27.8 x 35 mm
Changed lines of the file:
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@@
 		(tags "capacitor")
 		(property "Reference" "C12"
-			(at 0 -1.43 90)
+			(at -1.3 -1.45 90)
 			(layer "F.SilkS")
 			(effects
@@
 		)
 	)
+	(gr_rect
+		(start 99.75 105)
+		(end 127.5 140)
+		(stroke
+			(width 0.05)
+			(type default)
+		)
+		(fill no)
+		(layer "Edge.Cuts")
+	)
+	(segment
+		(start 114 110)
+		(end 113.25 110)
+		(width 0.4)
+		(layer "F.Cu")
+		(net "GND")
+	)
+	(via
+		(at 113.25 110)
+		(size 0.6)
+		(drill 0.3)
+		(layers "F.Cu" "B.Cu")
+		(net "GND")
+	)
 	(segment
 		(start 109.2 114.8)
@@
 	)
 	(segment
+		(start 124.075 124.025)
+		(end 114.905 124.025)
+		(width 0.2)
+		(layer "F.Cu")
+		(net "/MOSI")
+	)
+	(segment
 		(start 119.4 111.5)
 		(end 118.55 110.65)
@@
 	)
 	(segment
-		(start 119.9 118.2)
-		(end 116.4 121.7)
-		(width 0.2)
-		(layer "F.Cu")
-		(net "/MOSI")
-	)
-	(segment
-		(start 116.4 122.53)
-		(end 114.905 124.025)
-		(width 0.2)
-		(layer "F.Cu")
-		(net "/MOSI")
-	)
-	(segment
-		(start 116.4 121.7)
-		(end 116.4 122.53)
+		(start 125.38 122.72)
+		(end 124.075 124.025)
 		(width 0.2)
 		(layer "F.Cu")
@@
 		(net "/MOSI")
 	)
-	(via
-		(at 119.9 118.2)
-		(size 0.6)
-		(drill 0.3)
-		(layers "F.Cu" "B.Cu")
-		(net "/MOSI")
-	)
 	(segment
 		(start 119.9 118.2)
@@
 	)
 	(segment
-		(start 119.1 115)
-		(end 117.7 115)
+		(start 116.45 113.75)
+		(end 114 111.3)
 		(width 0.2)
 		(layer "F.Cu")
@@
 		(start 112.365 129.565)
 		(end 112.365 128.975)
+		(width 0.2)
+		(layer "F.Cu")
+		(net "/MISO")
+	)
+	(segment
+		(start 119.1 113.75)
+		(end 116.45 113.75)
 		(width 0.2)
 		(layer "F.Cu")
@@
 		(net "/MISO")
 	)
-	(segment
-		(start 117.7 115)
-		(end 114 111.3)
-		(width 0.2)
-		(layer "F.Cu")
-		(net "/MISO")
-	)
 	(via
-		(at 119.1 115)
+		(at 119.1 113.75)
 		(size 0.6)
 		(drill 0.3)
@@
 	)
 	(segment
+		(start 119.1 113.75)
+		(end 119.1 120.6)
+		(width 0.2)
+		(layer "B.Cu")
+		(net "/MISO")
+	)
+	(segment
+		(start 119.1 120.6)
+		(end 123.76 125.26)
+		(width 0.2)
+		(layer "B.Cu")
+		(net "/MISO")
+	)
+	(segment
 		(start 123.76 125.26)
-		(end 119.1 120.6)
-		(width 0.2)
-		(layer "B.Cu")
-		(net "/MISO")
-	)
-	(segment
-		(start 125.38 125.26)
-		(end 123.76 125.26)
-		(width 0.2)
-		(layer "B.Cu")
-		(net "/MISO")
-	)
-	(segment
-		(start 119.1 120.6)
-		(end 119.1 115)
+		(end 125.38 125.26)
 		(width 0.2)
 		(layer "B.Cu")
@@
 	(zone
 		(net "GND")
-		(layer "F.Cu")
+		(layers "F.Cu" "B.Cu")
 		(hatch edge 0.5)
 		(connect_pads
@@
 		)
 		(min_thickness 0.25)
-		(fill
+		(fill yes
 			(thermal_gap 0.5)
 			(thermal_bridge_width 0.5)
@@
 		(polygon
 			(pts
-				(xy 130 100) (xy 130 142) (xy 86 142) (xy 86 100)
-			)
-		)
-	)
-	(zone
-		(net "GND")
-		(layer "B.Cu")
-		(hatch edge 0.5)
-		(priority 1)
-		(connect_pads
-			(clearance 0.5)
-		)
-		(min_thickness 0.25)
-		(fill
-			(thermal_gap 0.5)
-			(thermal_bridge_width 0.5)
-			(island_removal_mode 0)
-		)
-		(polygon
-			(pts
-				(xy 130 142) (xy 130 100) (xy 86 100) (xy 86 142)
-			)
-		)
+				(xy 127.5 140) (xy 127.5 105) (xy 93 105) (xy 93.013202 140.013003)
+			)
+		)

Commit message: prosze aby nie było konlfikut panie Bożę danke
Parts:
- removed J4: Conn_01x08, Connector_PinHeader_2.54mm:PinHeader_1x08_P2.54mm_Vertical
- removed J5: Conn_01x10, Connector_PinHeader_2.54mm:PinHeader_1x10_P2.54mm_Vertical
- added J1: Conn_02x12_Odd_Even, Connector_PinSocket_2.54mm:PinSocket_2x12_P2.54mm_Vertical, F.Cu at (145.7, 129.5)
- added J2: Conn_02x12_Odd_Even, Connector_PinSocket_2.54mm:PinSocket_2x12_P2.54mm_Vertical, F.Cu at (145.7, 101.5)
- R2: renamed from R7; moved to F.Cu
- moved R2 66.8 mm to (175.5, 115.0), turned to -90 degrees
- moved C2 63.0 mm to (171.2, 113.2), turned to -90 degrees
- moved R1 61.1 mm to (173.5, 115.0)
- moved U2 54.5 mm to (166.6, 116.9), turned to 0 degrees
- moved C1 39.2 mm to (151.0, 114.2), turned to 180 degrees
- moved U1 36.6 mm to (151.0, 116.8)
- moved C3 35.9 mm to (147.8, 118.0), turned to 0 degrees
- renumbered C12 to C1, C13 to C2, C14 to C3, R6 to R1, U5 to U1, U6 to U2
Routing:
- net +3.3V: track 54.2 -> 69.0 mm, vias 1 -> 2
- net Net-(U2-~{WP}): track 6.00 -> 19.4 mm, vias 1 -> 2
- net /CS FRAM SPI: track 16.5 -> 27.9 mm, vias 0 -> 1
- net /CS BME280: track 25.8 -> 16.0 mm
- net /MISO: track 39.4 -> 31.6 mm
- net GND: track 0.75 -> 5.67 mm, vias 1 -> 0
- net Net-(U2-~{HOLD}): track 6.84 -> 4.60 mm
- net /MOSI: track 30.2 -> 30.3 mm, vias 1 -> 0
Other:
- board size 27.8 x 35 mm -> 37.5 x 35.5 mm
