File: czujnik/czujnik.kicad_sch (KiCad schematic)
At the start: 9 parts, among them J4 Conn_01x08, J5 Conn_01x10, U5 BME280, U6 MB85RS256B

Commit message: awetg2
Connections:
- net CS BME280: now also J4.7 (Pin_7); no longer J4.2 (Pin_2)
- net CS FRAM SPI: now also J4.8 (Pin_8); no longer J4.3 (Pin_3)
- net SCL: now also J4.3 (Pin_3); no longer J4.8 (Pin_8)
- net SDA: now also J4.2 (Pin_2); no longer J4.7 (Pin_7)

Commit message: czujnik pcb
Connections:
- net SCL: now also J4.2 (Pin_2); no longer J4.3 (Pin_3)
- net SDA: now also J4.3 (Pin_3); no longer J4.2 (Pin_2)
Changed lines of the file:
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@@
 		)
 	)
-	(label "SDA"
+	(label "SCL"
 		(at 173.99 66.04 180)
 		(effects
@@
 		)
 	)
-	(label "SCL"
+	(label "SDA"
 		(at 173.99 68.58 180)
 		(effects

Commit message: :3
Changed lines of the file:
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@@
+	)
+	(symbol
+		(lib_id "power:GNDREF")
+		(at 191.77 86.36 90)
+		(unit 1)
+		(body_style 1)
+		(exclude_from_sim no)
+		(in_bom yes)
+		(on_board yes)
+		(in_pos_files yes)
+		(dnp no)
+		(fields_autoplaced yes)
+		(property "Reference" "#PWR01"
+			(at 198.12 86.36 0)
+			(hide yes)
+			(show_name no)
+			(do_not_autoplace no)
+			(effects
+				(font
+					(size 1.27 1.27)
+				)
+			)
+		)
+		(property "Value" "GNDREF"
+			(at 195.58 86.3599 90)
+			(show_name no)
+			(do_not_autoplace no)
+			(effects
+				(font
+					(size 1.27 1.27)
+				)
+				(justify right)
+			)
+		)
+		(property "Footprint" ""
+			(at 191.77 86.36 0)
+			(hide yes)
+			(show_name no)
+			(do_not_autoplace no)
+			(effects
+				(font
+					(size 1.27 1.27)
+				)
+			)
+		)
+		(property "Datasheet" ""
+			(at 191.77 86.36 0)
+			(hide yes)
+			(show_name no)
+			(do_not_autoplace no)
+			(effects
+				(font
+					(size 1.27 1.27)
+				)
+			)
+		)
+		(property "Description" "Power symbol creates a global label with name \"GNDREF\" , reference supply ground"
+			(at 191.77 86.36 0)
+			(hide yes)
+			(show_name no)
+			(do_not_autoplace no)
+			(effects
+				(font
+					(size 1.27 1.27)
+				)
+			)
+		)
+		(pin "1"
+		)
+		(instances
+			(project "czujnik"
+				(path "/03e94da1-5877-4847-9c1a-1f6bf95d54b4"
+					(reference "#PWR01")
+					(unit 1)
+				)
+			)
+		)
 	)
 	(symbol

Commit message: Zmianakonnektora
Parts:
- removed J4: Conn_01x08, Connector_PinHeader_2.54mm:PinHeader_1x08_P2.54mm_Vertical, symbol Connector_Generic:Conn_01x08
- removed J5: Conn_01x10, Connector_PinHeader_2.54mm:PinHeader_1x10_P2.54mm_Vertical, symbol Connector_Generic:Conn_01x10
- added J6, J7: Conn_02x12_Odd_Even, Connector_PinSocket_2.54mm:PinSocket_2x12_P2.54mm_Vertical, symbol Connector_Generic:Conn_02x12_Odd_Even
Connections:
- net +3.3V: now also J6.1 (Pin_1), J6.2 (Pin_2), J7.1 (Pin_1), J7.3 (Pin_3)
- net COL 1: now also J6.4 (Pin_4)
- net COL 2: now also J6.6 (Pin_6)
- net COL 3: now also J6.8 (Pin_8)
- net COL 4: now also J6.10 (Pin_10)
- net CS BME280: now also J6.13 (Pin_13)
- net CS FRAM SPI: now also J6.15 (Pin_15)
- net GND: now also J6.19 (Pin_19), J6.20 (Pin_20), J6.21 (Pin_21), J6.22 (Pin_22), J6.23 (Pin_23), J6.24 (Pin_24), J7.15 (Pin_15), J7.17 (Pin_17), J7.19 (Pin_19), J7.21 (Pin_21), J7.23 (Pin_23)
- net MISO: now also J6.9 (Pin_9)
- net MOSI: now also J6.7 (Pin_7)
- net ROW 1: now also J6.12 (Pin_12)
- net ROW 2: now also J6.14 (Pin_14)
- net ROW 3: now also J6.16 (Pin_16)
- net ROW 4: now also J6.18 (Pin_18)
- net SCK: now also J6.11 (Pin_11)
- net SCL: now also J6.3 (Pin_3)
- net SDA: now also J6.5 (Pin_5)
- new net GPIO21: J7.5 (Pin_5)
- new net GPIO3: J6.17 (Pin_17)
- new net GPIO33: J7.10 (Pin_10)
- new net GPIO34: J7.12 (Pin_12)
- new net GPIO35: J7.14 (Pin_14)
- new net GPIO36: J7.16 (Pin_16)
- new net GPIO37: J7.18 (Pin_18)
- new net GPIO38: J7.20 (Pin_20)
- new net GPIO45: J7.22 (Pin_22)
- new net GPIO46: J7.24 (Pin_24)
- new net MTCK: J7.2 (Pin_2)
- new net MTDI: J7.6 (Pin_6)
- new net MTDO: J7.4 (Pin_4)
- new net MTMS: J7.8 (Pin_8)
- new net SPICLK_N: J7.13 (Pin_13)
- new net SPICLK_P: J7.11 (Pin_11)
- new net XTAL_32K_N: J7.9 (Pin_9)
- new net XTAL_32K_P: J7.7 (Pin_7)

Commit message: Zmianakonnektorav2
Parts:
- removed J7: Conn_02x12_Odd_Even, Connector_PinSocket_2.54mm:PinSocket_2x12_P2.54mm_Vertical, symbol Connector_Generic:Conn_02x12_Odd_Even
- added J4: Conn_02x12_Odd_Even, Connector_PinSocket_2.54mm:PinSocket_2x12_P2.54mm_Vertical, symbol Connector_Generic:Conn_02x12_Odd_Even
Connections:
- net +3.3V: now also J4.1 (Pin_1), J4.2 (Pin_2)
- net GND: now also J4.15 (Pin_15), J4.17 (Pin_17), J4.19 (Pin_19), J4.21 (Pin_21), J4.23 (Pin_23)
- net GPIO21: now also J4.5 (Pin_5)
- net GPIO33: now also J4.10 (Pin_10)
- net GPIO34: now also J4.12 (Pin_12)
- net GPIO35: now also J4.14 (Pin_14)
- net GPIO36: now also J4.16 (Pin_16)
- net GPIO37: now also J4.18 (Pin_18)
- net GPIO38: now also J4.20 (Pin_20)
- net GPIO45: now also J4.22 (Pin_22)
- net GPIO46: now also J4.24 (Pin_24)
- net MTCK: now also J4.3 (Pin_3)
- net MTDI: now also J4.6 (Pin_6)
- net MTDO: now also J4.4 (Pin_4)
- net MTMS: now also J4.8 (Pin_8)
- net SPICLK_N: now also J4.13 (Pin_13)
- net SPICLK_P: now also J4.11 (Pin_11)
- net XTAL_32K_N: now also J4.9 (Pin_9)
- net XTAL_32K_P: now also J4.7 (Pin_7)

Commit message: prosze aby nie było konlfikut panie Bożę danke
Parts:
- removed J4, J6: Conn_02x12_Odd_Even, Connector_PinSocket_2.54mm:PinSocket_2x12_P2.54mm_Vertical, symbol Connector_Generic:Conn_02x12_Odd_Even
- added J1, J2: Conn_02x12_Odd_Even, Connector_PinSocket_2.54mm:PinSocket_2x12_P2.54mm_Vertical, symbol Connector_Generic:Conn_02x12_Odd_Even
- renumbered C12 to C1, C13 to C2, C14 to C3, R6 to R1, R7 to R2, U5 to U1, U6 to U2
Connections:
- net +3.3V: now also J1.1 (Pin_1), J1.2 (Pin_2), J2.1 (Pin_1), J2.2 (Pin_2)
- net COL 1: now also J1.4 (Pin_4)
- net COL 2: now also J1.6 (Pin_6)
- net COL 3: now also J1.8 (Pin_8)
- net COL 4: now also J1.10 (Pin_10)
- net CS BME280: now also J1.5 (Pin_5)
- net CS FRAM SPI: now also J1.3 (Pin_3)
- net GND: now also J1.19 (Pin_19), J1.20 (Pin_20), J1.21 (Pin_21), J1.22 (Pin_22), J1.23 (Pin_23), J1.24 (Pin_24), J2.15 (Pin_15), J2.17 (Pin_17), J2.19 (Pin_19), J2.21 (Pin_21), J2.23 (Pin_23)
- net GPIO21: now also J2.5 (Pin_5)
- net GPIO3: now also J1.7 (Pin_7)
- net GPIO33: now also J2.10 (Pin_10)
- net GPIO34: now also J2.12 (Pin_12)
- net GPIO35: now also J2.14 (Pin_14)
- net GPIO36: now also J2.16 (Pin_16)
- net GPIO37: now also J2.18 (Pin_18)
- net GPIO38: now also J2.20 (Pin_20)
- net GPIO45: now also J2.22 (Pin_22)
- net GPIO46: now also J2.24 (Pin_24)
- net MISO: now also J1.11 (Pin_11)
- net MOSI: now also J1.13 (Pin_13)
- net MTCK: now also J2.3 (Pin_3)
- net MTDI: now also J2.6 (Pin_6)
- net MTDO: now also J2.4 (Pin_4)
- net MTMS: now also J2.8 (Pin_8)
- net ROW 1: now also J1.12 (Pin_12)
- net ROW 2: now also J1.14 (Pin_14)
- net ROW 3: now also J1.16 (Pin_16)
- net ROW 4: now also J1.18 (Pin_18)
- net SCK: now also J1.9 (Pin_9)
- net SCL: now also J1.17 (Pin_17)
- net SDA: now also J1.15 (Pin_15)
- net SPICLK_N: now also J2.13 (Pin_13)
- net SPICLK_P: now also J2.11 (Pin_11)
- net XTAL_32K_N: now also J2.9 (Pin_9)
- net XTAL_32K_P: now also J2.7 (Pin_7)
