File: wyświetlacz/wyświetlacz.kicad_pcb (KiCad board)
At the start: 2 copper layers, 9 parts, among them J8 Conn_01x08, J9 Conn_01x10, U7 MB85RC256V, U8 SSD1306

Commit message: :3
Parts:
- moved J9 56.3 mm to (167.2, 73.0)
- moved U7 51.2 mm to (145.1, 68.2)
- moved J8 39.1 mm to (149.4, 99.9), turned to 90 degrees
- moved C15 33.4 mm to (150.8, 65.4), turned to -90 degrees
- moved U8 28.0 mm to (124.9, 88.9), turned to 90 degrees
- moved R11 20.5 mm to (109.1, 71.6), turned to 180 degrees
- moved R10 15.2 mm to (109.1, 76.0), turned to 180 degrees
- moved R8 12.4 mm to (108.7, 85.7), turned to 180 degrees
- moved R9 11.6 mm to (109.0, 80.9), turned to 180 degrees

Commit message: prosze aby nie było konlfikut panie Bożę danke
Parts:
- removed C15: 100nF, Capacitor_SMD:C_0603_1608Metric
- removed J8: Conn_01x08, Connector_PinHeader_2.54mm:PinHeader_1x08_P2.54mm_Vertical
- removed J9: Conn_01x10, Connector_PinHeader_2.54mm:PinHeader_1x10_P2.54mm_Vertical
- removed R10, R11, R8, R9: 10k, Resistor_SMD:R_0603_1608Metric
- removed U7: MB85RC256V, Package_SO:SOIC-8_3.9x4.9mm_P1.27mm
- removed U8: SSD1306, Display:ER_OLEDM0.91_1x-I2C
- added C1: 100nF, Capacitor_SMD:C_0603_1608Metric, F.Cu at (132.3, 82.9)
- added C2: 100nF, Capacitor_SMD:C_0603_1608Metric, F.Cu at (131.8, 74.0)
- added J1: Conn_02x12_Odd_Even, Connector_PinSocket_2.54mm:PinSocket_2x12_P2.54mm_Vertical, F.Cu at (142.1, 86.5)
- added J2: Conn_02x12_Odd_Even, Connector_PinSocket_2.54mm:PinSocket_2x12_P2.54mm_Vertical, F.Cu at (142.1, 58.5)
- added R1: 10k, Resistor_SMD:R_0603_1608Metric, F.Cu at (125.8, 79.0)
- added R2: 10k, Resistor_SMD:R_0603_1608Metric, F.Cu at (127.5, 79.0)
- added R3: 10k, Resistor_SMD:R_0603_1608Metric, F.Cu at (124.0, 79.0)
- added R4: 10k, Resistor_SMD:R_0603_1608Metric, F.Cu at (129.2, 79.0)
- added U1: MB85RC256V, Package_SO:SOIC-8_3.9x4.9mm_P1.27mm, F.Cu at (127.5, 86.4)
- added U2: SSD1306, Display:ER_OLEDM0.91_1x-I2C, F.Cu at (135.2, 77.6)
Routing:
- net +3.3V: track 0.00 -> 58.6 mm
- net /SDA: track 0.00 -> 43.1 mm, vias 0 -> 1
- net /SCL: track 0.00 -> 34.6 mm, vias 0 -> 1
- net Net-(U1-A2): track 0.00 -> 8.92 mm
- net Net-(U1-WP): track 0.00 -> 7.84 mm
- net Net-(U1-A1): track 0.00 -> 7.51 mm
- net Net-(U1-A0): track 0.00 -> 4.94 mm
- added copper zone on B.Cu, net GND
- added copper zone on F.Cu, net GND
Other:
- board outline added: 57.2 x 37.5 mm
- copper layers 2 -> 4
