File: wyświetlacz/wyświetlacz.kicad_sch (KiCad schematic)
At the start: 9 parts, among them J8 Conn_01x08, J9 Conn_01x10, U7 MB85RC256V, U8 SSD1306

Commit message: :3
Connections:
- net CS BME280: now also J8.7 (Pin_7); no longer J8.2 (Pin_2)
- net CS FRAM SPI: now also J8.8 (Pin_8); no longer J8.3 (Pin_3)
- net SCL: now also J8.2 (Pin_2); no longer J8.8 (Pin_8)
- net SDA: now also J8.3 (Pin_3); no longer J8.7 (Pin_7)
Changed lines of the file:
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@@
-		)
-	)
-	(label "CS FRAM SPI"
-		(at 205.74 44.45 180)
-		(effects
-			(font
-				(size 1.27 1.27)
-			)
-			(justify right bottom)
 		)
 	)
@@
 		)
 	)
+	(label "SCL"
+		(at 205.74 41.91 180)
+		(effects
+			(font
+				(size 1.27 1.27)
+			)
+			(justify right bottom)
+		)
+	)
+	(label "SDA"
+		(at 205.74 44.45 180)
+		(effects
+			(font
+				(size 1.27 1.27)
+			)
+			(justify right bottom)
+		)
+	)
 	(label "MOSI"
 		(at 205.74 46.99 180)
@@
 		)
 	)
-	(label "SDA"
+	(label "CS BME280"
 		(at 205.74 54.61 180)
 		(effects
@@
 		)
 	)
-	(label "SCL"
+	(label "CS FRAM SPI"
 		(at 205.74 57.15 180)
 		(effects
@@
 			)
 			(justify left bottom)
-		)
-	)
-	(label "CS BME280"
-		(at 205.74 41.91 180)
-		(effects
-			(font
-				(size 1.27 1.27)
-			)
-			(justify right bottom)
 		)
 	)
@@
 		)
 		(instances
+			(project "wyświetlacz"
+				(path "/a85aa644-c8c0-48f2-bd06-479bc968afde"
+					(reference "#PWR034")
+					(unit 1)
+				)
+			)
 			(project "Projekt_smiw"
 				(path "/d5cd91f9-1e43-4778-a798-2ad13ae8c439"
@@
 		)
 		(instances
+			(project "wyświetlacz"
+				(path "/a85aa644-c8c0-48f2-bd06-479bc968afde"
+					(reference "#PWR036")
+					(unit 1)
+				)
+			)
 			(project "Projekt_smiw"
 				(path "/d5cd91f9-1e43-4778-a798-2ad13ae8c439"
@@
 		)
 		(instances
+			(project "wyświetlacz"
+				(path "/a85aa644-c8c0-48f2-bd06-479bc968afde"
+					(reference "R8")
+					(unit 1)
+				)
+			)
 			(project "Projekt_smiw"
 				(path "/d5cd91f9-1e43-4778-a798-2ad13ae8c439"
@@
 		)
 		(instances
+			(project "wyświetlacz"
+				(path "/a85aa644-c8c0-48f2-bd06-479bc968afde"
+					(reference "U8")
+					(unit 1)
+				)
+			)
 			(project "Projekt_smiw"
 				(path "/d5cd91f9-1e43-4778-a798-2ad13ae8c439"
@@
 		)
 		(instances
+			(project "wyświetlacz"
+				(path "/a85aa644-c8c0-48f2-bd06-479bc968afde"
+					(reference "#PWR035")
+					(unit 1)
+				)
+			)
 			(project "Projekt_smiw"
 				(path "/d5cd91f9-1e43-4778-a798-2ad13ae8c439"
@@
 		)
 		(instances
+			(project "wyświetlacz"
+				(path "/a85aa644-c8c0-48f2-bd06-479bc968afde"
+					(reference "#PWR031")
+					(unit 1)
+				)
+			)
 			(project "Projekt_smiw"
 				(path "/d5cd91f9-1e43-4778-a798-2ad13ae8c439"
@@
 		)
 		(instances
+			(project "wyświetlacz"
+				(path "/a85aa644-c8c0-48f2-bd06-479bc968afde"
+					(reference "#PWR033")
+					(unit 1)
+				)
+			)
 			(project "Projekt_smiw"
 				(path "/d5cd91f9-1e43-4778-a798-2ad13ae8c439"
@@
 		)
 		(instances
+			(project "wyświetlacz"
+				(path "/a85aa644-c8c0-48f2-bd06-479bc968afde"
+					(reference "J9")
+					(unit 1)
+				)
+			)
 			(project "Projekt_smiw"
 				(path "/d5cd91f9-1e43-4778-a798-2ad13ae8c439"
@@
 		)
 		(instances
+			(project "wyświetlacz"
+				(path "/a85aa644-c8c0-48f2-bd06-479bc968afde"
+					(reference "J8")
+					(unit 1)
+				)
+			)
 			(project "Projekt_smiw"
 				(path "/d5cd91f9-1e43-4778-a798-2ad13ae8c439"
@@
 		)
 		(instances
+			(project "wyświetlacz"
+				(path "/a85aa644-c8c0-48f2-bd06-479bc968afde"
+					(reference "R9")
+					(unit 1)
+				)
+			)
 			(project "Projekt_smiw"
 				(path "/d5cd91f9-1e43-4778-a798-2ad13ae8c439"
@@
 		)
 		(instances
+			(project "wyświetlacz"
+				(path "/a85aa644-c8c0-48f2-bd06-479bc968afde"
+					(reference "R10")
+					(unit 1)
+				)
+			)
 			(project "Projekt_smiw"
 				(path "/d5cd91f9-1e43-4778-a798-2ad13ae8c439"
@@
 		)
 		(instances
+			(project "wyświetlacz"
+				(path "/a85aa644-c8c0-48f2-bd06-479bc968afde"
+					(reference "C15")
+					(unit 1)
+				)
+			)
 			(project "Projekt_smiw"
 				(path "/d5cd91f9-1e43-4778-a798-2ad13ae8c439"
@@
 		)
 		(instances
+			(project "wyświetlacz"
+				(path "/a85aa644-c8c0-48f2-bd06-479bc968afde"
+					(reference "U7")
+					(unit 1)
+				)
+			)
 			(project "Projekt_smiw"
 				(path "/d5cd91f9-1e43-4778-a798-2ad13ae8c439"
@@
 		)
 		(instances
+			(project "wyświetlacz"
+				(path "/a85aa644-c8c0-48f2-bd06-479bc968afde"
+					(reference "#PWR032")
+					(unit 1)
+				)
+			)
 			(project "Projekt_smiw"
 				(path "/d5cd91f9-1e43-4778-a798-2ad13ae8c439"
@@
 		)
 		(instances
+			(project "wyświetlacz"
+				(path "/a85aa644-c8c0-48f2-bd06-479bc968afde"
+					(reference "R11")
+					(unit 1)
+				)
+			)
 			(project "Projekt_smiw"
 				(path "/d5cd91f9-1e43-4778-a798-2ad13ae8c439"
@@
 	)
 	(group "conn"
-		(members "03153902-e15d-4334-8f08-8eb4e10839b8" "0eb03138-6980-4ff7-810a-0ffa65b82c27"
-			"1440acc5-9798-46d5-b309-68ee94385d69" "15995232-5adc-4471-b7e8-b078319d211e"
-			"15bcd4b6-2e1f-4223-a590-718acde2d6ee" "236c41c1-10c7-4ac8-ad7d-30609b42287d"
-			"26e1143a-7c1b-48c4-b733-8f4192b23157" "2c70b218-4db1-4412-ab7f-98850486ddcf"
-			"320cb200-7b4b-41de-bcb9-0296de37bb91" "3427defa-3712-4057-bc17-aa233e7be427"
-			"35e96612-090d-4543-942a-91f0965a61e2" "393b176d-6fcc-4f85-9957-ab326870a822"
-			"3b5fc433-c742-4f12-926a-24d45c2710a5" "4107bc6c-f621-40e1-8653-ace4892797f0"
-			"41523854-2de1-4947-82e1-faf6d677a141" "425c6eb8-d8d3-4b34-8397-2c5972bce03e"
-			"508e9f0a-f316-4259-a61c-24a33109cdda" "5734570b-b760-4e66-96e5-12a6810da34d"
-			"57e00876-4017-48b3-979c-7dee161e0bcd" "5e81828b-e9b0-4ec9-bf3c-5515c72c985c"
-			"5f08a674-7e91-4bfd-9008-6387e86e5fb9" "6ad1988a-60ec-4fa4-ae7a-06db5b36d992"
-			"6c13ce2b-1ecd-49cb-bb8f-896598614149" "83e1c29a-b674-466e-ba5a-fff95532b66d"
-			"8b37eaf2-e042-480e-b278-a89636a31975" "8bbc6e05-0527-412c-ac2b-927e147c66c0"
-			"95913eb3-d73c-4136-abfa-1f8217abea73" "95bdf457-0f94-4786-993d-26e574e3e586"
-			"9645d19a-a170-4071-b56f-a309f7da7662" "a4534d7f-f130-4a5c-992e-142b11407aba"
-			"a53f8c8c-0abd-424a-bb87-4fe9ff88665b" "a6adbf17-e335-47bf-b023-b1fd5ccba0df"
+		(members "0eb03138-6980-4ff7-810a-0ffa65b82c27" "1440acc5-9798-46d5-b309-68ee94385d69"
+			"15995232-5adc-4471-b7e8-b078319d211e" "15bcd4b6-2e1f-4223-a590-718acde2d6ee"
+			"1b65644a-eeb7-42a3-a6b5-c9cefd5b9e16" "1c7af0d7-e38e-4d28-a86a-d8241c081806"
+			"236c41c1-10c7-4ac8-ad7d-30609b42287d" "26e1143a-7c1b-48c4-b733-8f4192b23157"
+			"2c70b218-4db1-4412-ab7f-98850486ddcf" "320cb200-7b4b-41de-bcb9-0296de37bb91"
+			"3427defa-3712-4057-bc17-aa233e7be427" "35e96612-090d-4543-942a-91f0965a61e2"
+			"393b176d-6fcc-4f85-9957-ab326870a822" "3b5fc433-c742-4f12-926a-24d45c2710a5"
+			"4107bc6c-f621-40e1-8653-ace4892797f0" "41523854-2de1-4947-82e1-faf6d677a141"
+			"425c6eb8-d8d3-4b34-8397-2c5972bce03e" "508e9f0a-f316-4259-a61c-24a33109cdda"
+			"50d17776-1f26-45fb-a260-2adb8423bb04" "57e00876-4017-48b3-979c-7dee161e0bcd"
+			"5e81828b-e9b0-4ec9-bf3c-5515c72c985c" "5f08a674-7e91-4bfd-9008-6387e86e5fb9"
+			"6ad1988a-60ec-4fa4-ae7a-06db5b36d992" "6c13ce2b-1ecd-49cb-bb8f-896598614149"
+			"724c581c-64b7-4e97-8448-29610291f1f7" "83e1c29a-b674-466e-ba5a-fff95532b66d"
+			"8bbc6e05-0527-412c-ac2b-927e147c66c0" "95913eb3-d73c-4136-abfa-1f8217abea73"
+			"95bdf457-0f94-4786-993d-26e574e3e586" "9645d19a-a170-4071-b56f-a309f7da7662"
+			"a4534d7f-f130-4a5c-992e-142b11407aba" "a6adbf17-e335-47bf-b023-b1fd5ccba0df"
 			"aa186c3e-c41a-48a9-bad2-870db3387964" "b2157496-772d-4819-9276-c32198dbcd68"
 			"b56ee0c8-bb28-498d-abfd-fb9f74f64ec9" "ca8fa204-a847-4cfc-8d12-506b39906e11"
@@
 		)
 	)
+	(embedded_fonts no)
 )

Commit message: Zmianakonnektora
Parts:
- removed J8: Conn_01x08, Connector_PinHeader_2.54mm:PinHeader_1x08_P2.54mm_Vertical, symbol Connector_Generic:Conn_01x08
- removed J9: Conn_01x10, Connector_PinHeader_2.54mm:PinHeader_1x10_P2.54mm_Vertical, symbol Connector_Generic:Conn_01x10
- added J4, J5: Conn_02x12_Odd_Even, Connector_PinSocket_2.54mm:PinSocket_2x12_P2.54mm_Vertical, symbol Connector_Generic:Conn_02x12_Odd_Even
Connections:
- net +3.3V: now also J4.1 (Pin_1), J4.3 (Pin_3), J5.1 (Pin_1), J5.2 (Pin_2)
- net COL 1: now also J5.4 (Pin_4)
- net COL 2: now also J5.6 (Pin_6)
- net COL 3: now also J5.8 (Pin_8)
- net COL 4: now also J5.10 (Pin_10)
- net CS BME280: now also J5.13 (Pin_13)
- net CS FRAM SPI: now also J5.15 (Pin_15)
- net GND: now also J4.15 (Pin_15), J4.17 (Pin_17), J4.19 (Pin_19), J4.21 (Pin_21), J4.23 (Pin_23), J5.19 (Pin_19), J5.20 (Pin_20), J5.21 (Pin_21), J5.22 (Pin_22), J5.23 (Pin_23), J5.24 (Pin_24)
- net MISO: now also J5.9 (Pin_9)
- net MOSI: now also J5.7 (Pin_7)
- net ROW 1: now also J5.12 (Pin_12)
- net ROW 2: now also J5.14 (Pin_14)
- net ROW 3: now also J5.16 (Pin_16)
- net ROW 4: now also J5.18 (Pin_18)
- net SCK: now also J5.11 (Pin_11)
- net SCL: now also J5.3 (Pin_3)
- net SDA: now also J5.5 (Pin_5)
- new net GPIO21: J4.5 (Pin_5)
- new net GPIO3: J5.17 (Pin_17)
- new net GPIO33: J4.10 (Pin_10)
- new net GPIO34: J4.12 (Pin_12)
- new net GPIO35: J4.14 (Pin_14)
- new net GPIO36: J4.16 (Pin_16)
- new net GPIO37: J4.18 (Pin_18)
- new net GPIO38: J4.20 (Pin_20)
- new net GPIO45: J4.22 (Pin_22)
- new net GPIO46: J4.24 (Pin_24)
- new net MTCK: J4.2 (Pin_2)
- new net MTDI: J4.6 (Pin_6)
- new net MTDO: J4.4 (Pin_4)
- new net MTMS: J4.8 (Pin_8)
- new net SPICLK_N: J4.13 (Pin_13)
- new net SPICLK_P: J4.11 (Pin_11)
- new net XTAL_32K_N: J4.9 (Pin_9)
- new net XTAL_32K_P: J4.7 (Pin_7)

Commit message: Zmianakonnektorav2
Connections:
- net +3.3V: now also J4.2 (Pin_2); no longer J4.3 (Pin_3)
- net MTCK: now also J4.3 (Pin_3); no longer J4.2 (Pin_2)

Commit message: prosze aby nie było konlfikut panie Bożę danke
Parts:
- added C2: 100nF, Capacitor_SMD:C_0603_1608Metric, symbol Device:C_Small
- renumbered C15 to C1, J5 to J1, J4 to J2, R8 to R1, R9 to R2, R10 to R3, R11 to R4, U7 to U1, U8 to U2
Connections:
- net +3.3V: now also C2.1
- net GND: now also C2.2
Other:
- moved on the sheet: C1, R1, R2, R3, R4, U1, U2
